File: source/foc.kicad_pcb (KiCad board)
At the start: 2 copper layers, 68 x 79 mm, 218 parts, among them J1 Conn_01x04_Male, J2 TYPE-C-31-M-12, P1 SWD, Q1 MMBT5401, Q10 CSD19536KCS, Q11 CSD19536KCS, Q12 CSD19536KCS, Q13 MMBT5401, Q14 MMBT5401, Q15 CSD19536KCS, Q16 CSD19536KCS, Q17 CSD19536KCS, Q18 CSD19536KCS, Q2 MMBT5401, Q3 NCEP60T20, Q4 CSD19536KCS, Q5 CSD19536KCS, Q6 CSD19536KCS, Q7 MMBT5401, Q8 MMBT5401, Q9 CSD19536KCS, U1 BMI160, U10 HT7550, U11 STM32F405RGT6, U12 AMS1117-3.3, U2 IRS21867S, U3 IRS21867S, U4 IRS21867S, U5 TX4130L/PW2902, U6 MS8311, U7 MS8311, U8 MS8311, U9 TJA1050T/CM,118, Y1 8MHz Crystal Resonator, X5032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

Commit message: Add files via upload
Parts:
- removed FieldFeets1: R, Custom:field
- added C39: 4.7n, Capacitor_SMD:C_0603_1608Metric, F.Cu at (80.8, 89.5)
- added C41: 4.7n, Capacitor_SMD:C_0603_1608Metric, F.Cu at (80.8, 92.5)
- added C61: 4.7n, Capacitor_SMD:C_0603_1608Metric, F.Cu at (103.4, 89.2)
- added C63: 4.7n, Capacitor_SMD:C_0603_1608Metric, F.Cu at (103.4, 92.1)
- added C82: 4.7n, Capacitor_SMD:C_0603_1608Metric, F.Cu at (125.0, 88.7)
- added C83: 4.7n, Capacitor_SMD:C_0603_1608Metric, F.Cu at (125.0, 91.6)
- added H1: MountingHole, MountingHole:MountingHole_3.2mm_M3, F.Cu at (63.1, 119.3)
- added H2: MountingHole, MountingHole:MountingHole_3.2mm_M3, F.Cu at (117.9, 113.2)
- added H3: MountingHole, MountingHole:MountingHole_3.2mm_M3, F.Cu at (124.7, 119.3)
- added H4: MountingHole, MountingHole:MountingHole_3.2mm_M3, F.Cu at (73.6, 113.2)
- added H5: MountingHole, MountingHole:MountingHole_3.2mm_M3, F.Cu at (93.2, 75.8)
- added H6: MountingHole, MountingHole:MountingHole_3.2mm_M3, F.Cu at (95.7, 113.2)
- added R31: 10R, Resistor_SMD:R_0603_1608Metric, F.Cu at (82.2, 95.5)
- added R32: 10R, Resistor_SMD:R_0603_1608Metric, F.Cu at (80.8, 95.5)
- added R45: 10R, Resistor_SMD:R_0603_1608Metric, F.Cu at (103.4, 95.1)
- added R46: 10R, Resistor_SMD:R_0603_1608Metric, F.Cu at (104.8, 95.1)
- added R57: 10R, Resistor_SMD:R_0603_1608Metric, F.Cu at (126.5, 94.6)
- added R58: 10R, Resistor_SMD:R_0603_1608Metric, F.Cu at (125.0, 94.6)
- moved R6 3.85 mm to (82.0, 82.0)
- moved R7 3.85 mm to (82.0, 79.1)
- moved C65 3.35 mm to (121.3, 114.0), turned to 180 degrees
- moved R9 1.74 mm to (104.8, 92.2)
- moved R8 1.72 mm to (104.8, 89.2)
- moved R12 1.45 mm to (126.5, 88.6)
- moved R13 1.45 mm to (126.5, 91.7)
- moved R3 1.30 mm to (82.2, 89.5)
- moved R4 1.30 mm to (82.2, 92.5)
- moved C3 1.05 mm to (62.7, 114.5)
- moved D1 0.65 mm to (62.9, 111.3)
- renumbered C98 to C100, C99 to C101, C101 to C103, C102 to C104, C103 to C105, C104 to C106, C105 to C107, C106 to C108, C107 to C109, C17 to C13, C18 to C14, C19 to C15, C20 to C16, C21 to C17, C22 to C18, C23 to C19, C24 to C20, C25 to C21, C26 to C22, C27 to C23, C28 to C24, C29 to C25, C30 to C26, C31 to C27, C32 to C28, C33 to C29, C34 to C30, C35 to C31, C36 to C32, C37 to C33, C38 to C34, C39 to C35, C40 to C36, C41 to C37, C42 to C38, C43 to C40, C44 to C42, C45 to C43, C47 to C45, C48 to C46, C49 to C47, C50 to C48, C51 to C49, C52 to C50, C53 to C51, C54 to C52, C55 to C53, C56 to C54, C57 to C55, C58 to C56, C59 to C57, C60 to C58, C61 to C59, C62 to C60, C64 to C62, C63 to C64, C82 to C84, C83 to C85, C84 to C86, C85 to C87, C86 to C88, C87 to C89, C88 to C90, C89 to C91, C90 to C92, C91 to C93, C93 to C94, C92 to C95, C94 to C96, C96 to C98, C97 to C99, R31 to R33, R33 to R35, R34 to R36, R35 to R37, R37 to R39, R38 to R40, R39 to R41, R40 to R42, R41 to R43, R42 to R44, R43 to R47, R44 to R48, R45 to R49, R46 to R50, R47 to R51, R48 to R52, R49 to R53, R50 to R54, R51 to R55, R52 to R56, R53 to R59, R54 to R60, R55 to R61, R56 to R62, R57 to R63, R58 to R64, R59 to R65
Routing:
- net Net-(C66-Pad1): track 32.8 -> 54.4 mm
- net Net-(C23-Pad1): track 32.9 -> 51.5 mm
- net GND: track 204.7 -> 212.6 mm, vias 161 -> 162
- net /driver/SENS_SUPPLY: track 52.3 -> 56.5 mm
- net Net-(C45-Pad1): track 33.1 -> 36.8 mm
- net Net-(C41-Pad2): track 0.00 -> 2.83 mm
- net Net-(C83-Pad2): track 0.00 -> 2.80 mm
- net Net-(C63-Pad2): track 0.00 -> 2.80 mm
- net VCC: track 169.9 -> 172.6 mm
- net V_IN: track 132.0 -> 134.6 mm
- net /driver/HS2: track 19.0 -> 20.9 mm
- net /driver/SENS_3: track 71.3 -> 73.1 mm
- net Net-(D14-Pad2): track 3.73 -> 5.46 mm
- net Net-(D10-Pad2): track 3.73 -> 5.46 mm
- net Net-(D12-Pad2): track 3.73 -> 5.46 mm
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Other:
- board text added: "A"
- board text added: "B"
- board text added: "C"
- board text added: "NEG"
- board text added: "POS"
- board text added: "VECTORWAVE"
- board text removed: "NORDSTREAM3"

Commit message: Add files via upload
Parts:
- added C44: 2.2u, Capacitor_SMD:C_0603_1608Metric, F.Cu at (77.8, 101.4)
- added R34: NTC 10k, Resistor_SMD:R_0603_1608Metric, F.Cu at (74.8, 103.5)
- added R38: 10k, Resistor_SMD:R_0603_1608Metric, F.Cu at (77.1, 103.7)
- moved R25 0.92 mm to (74.9, 105.7)
- moved R28 0.63 mm to (78.6, 105.1)
- moved R29 0.63 mm to (80.1, 105.1)
- moved C25 0.47 mm to (79.4, 102.9)
- moved H4 0.40 mm to (73.2, 113.2)
- moved U6 0.38 mm to (77.8, 108.7)
- moved R24 0.28 mm to (78.2, 111.5)
- moved R21 0.10 mm to (76.0, 112.0)
Routing:
- net /mcu/ADC_TEMP: track 0.00 -> 47.7 mm, vias 0 -> 8
- net GND: track 212.6 -> 214.9 mm, vias 162 -> 164
- net Net-(C25-Pad1): track 18.0 -> 18.6 mm
- net VCC: track 172.6 -> 173.3 mm
- net Net-(R25-Pad1): track 5.74 -> 6.34 mm
- net +12V: track 227.6 -> 228.1 mm
- added copper zone on B.Cu, net /mcu/ADC_TEMP
- added copper zone on F.Cu, net /mcu/ADC_TEMP

Commit message: Add files via upload
Parts:
- removed the C10 at (125.4, 122.8)
- removed the C26 at (63.5, 84.6)
- removed C28, C30, C32, C48, C59: 10u @ 50V, Capacitor_SMD:C_1206_3216Metric
- removed the C29 at (66.5, 79.6)
- removed the C33 at (72.5, 79.6)
- removed the C36 at (78.5, 84.6)
- removed the C37 at (78.5, 79.6)
- removed the C39 at (80.8, 89.5)
- removed the C51 at (88.5, 79.6)
- removed the C52 at (91.5, 84.6)
- removed the C54 at (94.5, 84.6)
- removed the C55 at (94.5, 79.6)
- removed the C56 at (97.5, 84.6)
- removed the C58 at (100.5, 84.6)
- removed C61: 4.7n, Capacitor_SMD:C_0603_1608Metric
- removed the C69 at (107.5, 84.7)
- removed the C71 at (110.5, 84.7)
- removed the C72 at (110.5, 79.7)
- removed the C73 at (113.5, 84.6)
- removed the C75 at (116.5, 84.7)
- removed the C76 at (116.5, 79.7)
- removed the C77 at (119.5, 84.6)
- removed the C79 at (122.5, 84.6)
- removed the C80 at (122.5, 79.6)
- removed the C82 at (125.0, 88.7)
- removed the D10 at (62.1, 108.7)
- removed the D11 at (70.6, 107.8)
- removed the D12 at (84.3, 108.7)
- removed D13, D14, D15: 1N4148WS, Diode_SMD:D_SOD-323
- removed the Q1 at (62.2, 105.8)
- removed Q13, Q14: MMBT5401, Package_TO_SOT_SMD:SOT-23
- removed the Q2 at (71.1, 104.9)
- removed the Q7 at (84.4, 105.8)
- removed the Q8 at (93.3, 104.9)
- added C3: 10u, Capacitor_Tantalum_SMD:CP_EIA-3216-10_Kemet-I, F.Cu at (63.4, 113.0)
- added C65: 4.7n, Capacitor_SMD:C_0603_1608Metric, F.Cu at (125.0, 88.7)
- added C8: 10u, Capacitor_Tantalum_SMD:CP_EIA-3216-10_Kemet-I, F.Cu at (86.1, 113.1)
- added H7: MountingHole, MountingHole:MountingHole_3.2mm_M3, F.Cu at (65.6, 75.8)
- added H8: MountingHole, MountingHole:MountingHole_3.7mm, F.Cu at (93.0, 76.0)
- added R31: 10R, Resistor_SMD:R_0603_1608Metric, F.Cu at (80.8, 86.5)
- added R33: 10R, Resistor_SMD:R_0603_1608Metric, F.Cu at (82.2, 86.5)
- added R47: 10R, Resistor_SMD:R_0603_1608Metric, F.Cu at (104.0, 86.2)
- added R49: 10R, Resistor_SMD:R_0603_1608Metric, F.Cu at (105.4, 86.2)
- added R61: 10R, Resistor_SMD:R_0603_1608Metric, F.Cu at (125.0, 85.7)
- added R63: 10R, Resistor_SMD:R_0603_1608Metric, F.Cu at (126.5, 85.7)
- C10: renamed from C8; value 100n -> 1u
- C11: renamed from C9; value 10u @ 50V -> 10u @ 100V; footprint Capacitor_SMD:C_1206_3216Metric -> Capacitor_SMD:C_2220_5650Metric
- C12: value 10u @ 50V -> 10u; footprint Capacitor_SMD:C_1206_3216Metric -> Capacitor_Tantalum_SMD:CP_EIA-3216-10_Kemet-I
- C13: renamed from C11; value 10u @ 50V -> 10u @ 100V; footprint Capacitor_SMD:C_1206_3216Metric -> Capacitor_SMD:C_2220_5650Metric
- C16: renamed from C15; value 100n -> 1u
- C27: value 10u @ 50V -> 10u @ 100V; footprint Capacitor_SMD:C_1206_3216Metric -> Capacitor_SMD:C_2220_5650Metric
- C29: renamed from C31; value 10u @ 50V -> 10u @ 100V; footprint Capacitor_SMD:C_1206_3216Metric -> Capacitor_SMD:C_2220_5650Metric
- C31: renamed from C35; value 10u @ 50V -> 10u @ 100V; footprint Capacitor_SMD:C_1206_3216Metric -> Capacitor_SMD:C_2220_5650Metric
- C34, C50: value 10u @ 50V -> 4.7n; footprint Capacitor_SMD:C_1206_3216Metric -> Capacitor_SMD:C_0603_1608Metric
- C43: renamed from C49; value 10u @ 50V -> 10u @ 100V; footprint Capacitor_SMD:C_1206_3216Metric -> Capacitor_SMD:C_2220_5650Metric
- C45: renamed from C53; value 10u @ 50V -> 10u @ 100V; footprint Capacitor_SMD:C_1206_3216Metric -> Capacitor_SMD:C_2220_5650Metric
- C47: renamed from C57; value 10u @ 50V -> 10u @ 100V; footprint Capacitor_SMD:C_1206_3216Metric -> Capacitor_SMD:C_2220_5650Metric
- C58: renamed from C70; value 10u @ 50V -> 10u @ 100V; footprint Capacitor_SMD:C_1206_3216Metric -> Capacitor_SMD:C_2220_5650Metric
- C6: renamed from C5; value 100n -> 1u
- C60: renamed from C74; value 10u @ 50V -> 10u @ 100V; footprint Capacitor_SMD:C_1206_3216Metric -> Capacitor_SMD:C_2220_5650Metric
- C62: renamed from C78; value 10u @ 50V -> 10u @ 100V; footprint Capacitor_SMD:C_1206_3216Metric -> Capacitor_SMD:C_2220_5650Metric
- H2, H4, H6: footprint MountingHole:MountingHole_3.2mm_M3 -> MountingHole:MountingHole_3.7mm
- moved C54 29.7 mm to (95.6, 128.8)
- moved H5 27.5 mm to (120.6, 75.8)
- moved C12 21.8 mm to (107.2, 113.2)
- moved R37 17.4 mm to (88.1, 94.5), turned to 0 degrees
- moved R52 17.4 mm to (110.3, 94.5), turned to 0 degrees
- moved R22 17.3 mm to (65.9, 94.5), turned to 0 degrees
- moved C38 17.2 mm to (85.8, 124.9), turned to 0 degrees
- moved C50 16.1 mm to (104.0, 89.2), turned to 90 degrees
- moved R56 12.6 mm to (114.5, 93.4), turned to 90 degrees
- moved C55 12.6 mm to (116.0, 93.4), turned to -90 degrees
- moved R42 12.6 mm to (92.3, 93.5), turned to 90 degrees
- moved C40 12.5 mm to (93.8, 93.5), turned to -90 degrees
- moved C24 12.4 mm to (71.5, 93.6), turned to -90 degrees
- moved R26 12.4 mm to (70.0, 93.6), turned to 90 degrees
- moved C90 8.36 mm to (77.0, 128.2), turned to 90 degrees
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- renumbered C13 to C14, C14 to C15, C16 to C17, C17 to C18, C18 to C19, C19 to C20, C20 to C21, C21 to C22, C22 to C23, C23 to C24, C24 to C25, C25 to C26, C38 to C33, C41 to C35, C40 to C36, C42 to C37, C43 to C38, C44 to C39, C3 to C4, C45 to C40, C46 to C41, C47 to C42, C60 to C49, C4 to C5, C63 to C51, C62 to C52, C64 to C53, C65 to C54, C66 to C55, C67 to C56, C68 to C57, C81 to C64, C83 to C66, C84 to C67, C85 to C68, C86 to C69, C6 to C7, C87 to C70, C88 to C71, C89 to C72, C90 to C73, C91 to C74, C92 to C75, C93 to C76, C94 to C77, C95 to C78, C96 to C79, C99 to C80, C98 to C81, C103 to C82, C100 to C83, C101 to C84, C104 to C85, C105 to C86, C106 to C87, C107 to C88, C108 to C89, C7 to C9, C109 to C90, D16 to D10, D17 to D11, D18 to D12, Q3 to Q1, Q16 to Q10, Q17 to Q11, Q18 to Q12, Q4 to Q2, Q5 to Q3, Q6 to Q4, Q9 to Q5, Q10 to Q6, Q11 to Q7, Q12 to Q8, Q15 to Q9, R31 to R32, R32 to R34, R33 to R35, R34 to R36, R35 to R37, R36 to R38, R37 to R39, R38 to R40, R39 to R41, R40 to R42, R41 to R43, R42 to R44, R43 to R45, R44 to R46, R45 to R48, R46 to R50, R47 to R51, R48 to R52, R49 to R53, R50 to R54, R51 to R55, R52 to R56, R53 to R57, R54 to R58, R55 to R59, R56 to R60, R57 to R62, R58 to R64, R59 to R65, R60 to R66, R61 to R67, R62 to R68, R63 to R69, R64 to R70, R65 to R71
Connections:
- C11 pad 1: Net-(C10-Pad2) (its old number) -> GND
- C12 pad 1: Net-(C11-Pad2) -> +12V
- C13 pad 2: Net-(C11-Pad2) -> GND
- C24 pad 1: Net-(C23-Pad1) -> Net-(C24-Pad1)
- C25 pad 1: Net-(C24-Pad1) -> Net-(C25-Pad1)
- C27 pad 2: Net-(C26-Pad1) (its old number) -> V_IN
- C29 pad 2: Net-(C30-Pad1) -> V_IN
- C31 pad 2: Net-(C34-Pad1) -> V_IN
- C34 pad 1: Net-(C34-Pad1) -> /driver/HS1
- C34 pad 2: V_IN -> Net-(C34-Pad2)
- C35 pad 1: Net-(C39-Pad1) -> /driver/HS1
- C40 pad 1: Net-(C45-Pad1) -> Net-(C40-Pad1)
- C41 pad 1: Net-(C46-Pad1) -> Net-(C41-Pad1)
- C43 pad 2: Net-(C48-Pad1) -> V_IN
- C45 pad 2: Net-(C52-Pad1) -> V_IN
- C47 pad 2: Net-(C56-Pad1) -> V_IN
- C50 pad 1: Net-(C50-Pad1) -> /driver/HS2
- C50 pad 2: V_IN -> Net-(C50-Pad2)
- C51 pad 1: Net-(C61-Pad1) -> /driver/HS2
- C55 pad 1: Net-(C66-Pad1) -> Net-(C55-Pad1)
- C56 pad 1: Net-(C67-Pad1) (its old number) -> Net-(C56-Pad1)
- C58 pad 2: Net-(C69-Pad1) -> V_IN
- C60 pad 2: Net-(C73-Pad1) -> V_IN
- C62 pad 2: Net-(C77-Pad1) -> V_IN
- C66 pad 1: Net-(C82-Pad1) -> /driver/HS3
- Q1 pad 1: Net-(C23-Pad1) -> Net-(C24-Pad1)
- Q10 pad 1: Net-(C67-Pad1) (its old number) -> Net-(C56-Pad1)
- Q11 pad 1: Net-(C66-Pad1) -> Net-(C55-Pad1)
- Q12 pad 1: Net-(C67-Pad1) (its old number) -> Net-(C56-Pad1)
- Q2 pad 1: Net-(C24-Pad1) -> Net-(C25-Pad1)
- Q3 pad 1: Net-(C23-Pad1) -> Net-(C24-Pad1)
- Q4 pad 1: Net-(C24-Pad1) -> Net-(C25-Pad1)
- Q5 pad 1: Net-(C45-Pad1) -> Net-(C40-Pad1)
- Q6 pad 1: Net-(C46-Pad1) -> Net-(C41-Pad1)
- Q7 pad 1: Net-(C45-Pad1) -> Net-(C40-Pad1)
- Q8 pad 1: Net-(C46-Pad1) -> Net-(C41-Pad1)
- Q9 pad 1: Net-(C66-Pad1) -> Net-(C55-Pad1)
- R22 pad 2: Net-(D10-Pad2) -> Net-(C24-Pad1)
- R23 pad 2: Net-(D11-Pad2) -> Net-(C25-Pad1)
- R26 pad 2: Net-(C23-Pad1) -> Net-(C24-Pad1)
- R27 pad 2: Net-(C24-Pad1) -> Net-(C25-Pad1)
- R37 pad 2: Net-(D12-Pad2) -> Net-(C40-Pad1)
- R38 pad 2: Net-(D13-Pad2) -> Net-(C41-Pad1)
- R42 pad 2: Net-(C45-Pad1) -> Net-(C40-Pad1)
- R43 pad 2: Net-(C46-Pad1) -> Net-(C41-Pad1)
- R52 pad 2: Net-(D14-Pad2) -> Net-(C55-Pad1)
- R53 pad 2: Net-(D15-Pad2) -> Net-(C56-Pad1)
- R56 pad 2: Net-(C66-Pad1) -> Net-(C55-Pad1)
- R57 pad 2: Net-(C67-Pad1) (its old number) -> Net-(C56-Pad1)
Routing:
- net Net-(C66-Pad1): track 54.4 -> 0.00 mm
- net Net-(C23-Pad1): track 51.5 -> 0.00 mm
- net V_IN: track 134.6 -> 86.1 mm
- net GND: track 214.9 -> 168.2 mm, vias 164 -> 185
- net Net-(C45-Pad1): track 36.8 -> 0.00 mm
- net VCC: track 173.3 -> 204.6 mm, vias 4 -> 7
- net +12V: track 228.1 -> 255.7 mm, vias 4 -> 8
- net Net-(C41-Pad1): track 0.00 -> 26.1 mm
- net Net-(C25-Pad1): track 0.00 -> 23.2 mm
- net Net-(C46-Pad1): track 22.3 -> 0.00 mm
- net Net-(C67-Pad1) (its old number): track 22.3 -> 0.00 mm
- net Net-(C40-Pad1): track 0.00 -> 21.5 mm
- net Net-(C55-Pad1): track 0.00 -> 21.4 mm
- net Net-(C56-Pad1): track 2.05 -> 20.7 mm
- net /driver/HO1: track 6.51 -> 19.9 mm
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Other:
- board size 68 x 79 mm -> 68.4 x 79 mm
- board text added: "WATT'EVER"
- board text removed: "VECTORWAVE"

Commit message: Add files via upload
Parts:
- removed the C21 at (73.7, 108.8)
- removed the C22 at (75.3, 108.8)
- removed the C26 at (79.4, 102.9)
- removed the C31 at (77.1, 83.3)
- removed the C33 at (78.2, 87.5)
- removed the C40 at (93.8, 93.5)
- removed the C41 at (93.6, 99.6)
- removed the C58 at (109.5, 83.0)
- removed the H2 at (115.2, 113.7)
- removed the H4 at (70.8, 113.7)
- removed H8: MountingHole, MountingHole:MountingHole_3.7mm
- removed Q10, Q11, Q12, Q7, Q8, Q9: CSD19536KCS, Package_TO_SOT_THT:TO-220-3_Vertical
- removed the R21 at (80.2, 112.2)
- removed the R24 at (80.2, 109.3)
- removed the R25 at (74.9, 105.7)
- removed the R28 at (78.6, 105.1)
- removed the R29 at (80.1, 105.1)
- removed the U6 at (77.8, 108.7)
- added C27: 100n 100V, Capacitor_SMD:C_0805_2012Metric, F.Cu at (75.5, 86.0)
- added C28: 100n 100V, Capacitor_SMD:C_0805_2012Metric, F.Cu at (65.3, 88.3)
- added C29: 100n 100V, Capacitor_SMD:C_0805_2012Metric, F.Cu at (65.3, 86.3)
- added C30: 100n 100V, Capacitor_SMD:C_0805_2012Metric, F.Cu at (65.3, 80.4)
- added C32: 100n 100V, Capacitor_SMD:C_0805_2012Metric, F.Cu at (65.3, 82.4)
- added C34: 100n 100V, Capacitor_SMD:C_0805_2012Metric, F.Cu at (65.3, 84.3)
- added C35: 470u 80V, Capacitor_THT:CP_Radial_D10.0mm_P5.00mm, F.Cu at (70.8, 69.5)
- added C38: 2.2u, Capacitor_SMD:C_0603_1608Metric, F.Cu at (94.6, 110.0)
- added C39: 100n, Capacitor_SMD:C_0603_1608Metric, F.Cu at (96.2, 110.0)
- added C42: 2.2nF, Capacitor_SMD:C_0603_1608Metric, F.Cu at (85.7, 95.7)
- added C44: 100p, Capacitor_SMD:C_0603_1608Metric, F.Cu at (98.6, 103.6)
- added C46: 100n 100V, Capacitor_SMD:C_0805_2012Metric, F.Cu at (83.2, 87.4)
- added C48: 100n 100V, Capacitor_SMD:C_0805_2012Metric, F.Cu at (83.2, 79.5)
- added C54: 4.7n, Capacitor_SMD:C_0603_1608Metric, F.Cu at (93.4, 86.8)
- added C59: 2.2nF, Capacitor_SMD:C_0603_1608Metric, F.Cu at (106.1, 95.7)
- added C61: 100p, Capacitor_SMD:C_0603_1608Metric, F.Cu at (117.8, 103.7)
- added C63: 100n 100V, Capacitor_SMD:C_0805_2012Metric, F.Cu at (103.5, 85.2)
- added C67: 100n 100V, Capacitor_SMD:C_0805_2012Metric, F.Cu at (103.5, 81.2)
- added C68: 10u @ 100V, Capacitor_SMD:C_2220_5650Metric, F.Cu at (118.6, 76.1)
- added C69: 100n 100V, Capacitor_SMD:C_0805_2012Metric, F.Cu at (103.5, 83.2)
- added C70: 470u 80V, Capacitor_THT:CP_Radial_D10.0mm_P5.00mm, F.Cu at (111.5, 69.5)
- added C71: 4.7n, Capacitor_SMD:C_0603_1608Metric, F.Cu at (113.8, 86.8)
- added C72: 4.7n, Capacitor_SMD:C_0603_1608Metric, F.Cu at (119.4, 88.8)
- added H3: MountingHole, MountingHole:MountingHole_3.2mm_M3, F.Cu at (93.8, 63.4)
- added H7: MountingHole_Pad, MountingHole:MountingHole_4mm_Pad_TopOnly, F.Cu at (87.0, 64.0)
- added R35: 30k, Resistor_SMD:R_0603_1608Metric, F.Cu at (101.1, 113.0)
- added R39: 30k, Resistor_SMD:R_0603_1608Metric, F.Cu at (101.1, 110.1)
- added R41: 62k, Resistor_SMD:R_0603_1608Metric, F.Cu at (96.2, 107.0)
- added R44: 1k, Resistor_SMD:R_0603_1608Metric, F.Cu at (97.9, 105.9)
- added R45: 1k, Resistor_SMD:R_0603_1608Metric, F.Cu at (99.4, 105.9)
- added U7: MS8311, Package_TO_SOT_SMD:TSOT-23-5, F.Cu at (98.7, 109.6)
- C43, C60: value 10u @ 100V -> 2.2nF; footprint Capacitor_SMD:C_2220_5650Metric -> Capacitor_SMD:C_0603_1608Metric
- C45, C47, C62: value 10u @ 100V -> 100n 100V; footprint Capacitor_SMD:C_2220_5650Metric -> Capacitor_SMD:C_0805_2012Metric
- C49: value 470u 80V -> 10u @ 100V; footprint Custom:CP_Radial_D8.0mm_P5.00mm -> Capacitor_SMD:C_2220_5650Metric
- C50, C65: value 4.7n -> 100n 100V; footprint Capacitor_SMD:C_0603_1608Metric -> Capacitor_SMD:C_0805_2012Metric
- C51, C66: value 4.7n -> 10u @ 100V; footprint Capacitor_SMD:C_0603_1608Metric -> Capacitor_SMD:C_2220_5650Metric
- C52: value 2.2u -> 100n 100V; footprint Capacitor_SMD:C_0603_1608Metric -> Capacitor_SMD:C_0805_2012Metric
- C53: value 100n -> 470u 80V; footprint Capacitor_SMD:C_0603_1608Metric -> Capacitor_THT:CP_Radial_D10.0mm_P5.00mm
- C55: value 2.2nF -> 4.7n
- C56: value 2.2nF -> 2.2u
- C57: value 100p -> 100n
- C64: value 470u 80V -> 100n 100V; footprint Custom:CP_Radial_D8.0mm_P5.00mm -> Capacitor_SMD:C_0805_2012Metric
- H6: value MountingHole -> MountingHole_Pad; footprint MountingHole:MountingHole_3.7mm -> MountingHole:MountingHole_4mm_Pad_TopOnly
- moved H6 50.3 mm to (101.0, 64.0)
- moved C53 48.2 mm to (91.1, 69.5), turned to 180 degrees
- moved C52 42.6 mm to (83.2, 83.4), turned to 180 degrees
- moved Q4 31.9 mm to (99.4, 92.9)
- moved Q6 30.1 mm to (119.8, 92.9)
- moved C26 23.6 mm to (78.3, 103.6)
- moved Q3 23.6 mm to (86.6, 91.0)
- moved C65 23.5 mm to (103.5, 79.2), turned to 180 degrees
- moved R28 23.1 mm to (77.6, 105.9)
- moved R29 23.1 mm to (79.1, 105.9)
- moved R25 22.5 mm to (75.9, 107.0), turned to -90 degrees
- moved C50 22.1 mm to (83.2, 81.4), turned to 180 degrees
- moved C21 21.9 mm to (74.2, 110.1)
- moved C22 21.9 mm to (75.8, 110.1)
- moved R21 21.9 mm to (80.8, 113.0)
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- renumbered C36 to C21, C37 to C22, C42 to C26, C27 to C31, C29 to C33, C34 to C36, C35 to C37, C38 to C40, C39 to C41, C54 to C58, C67 to C73, C68 to C74, C69 to C75, C70 to C76, C71 to C77, C72 to C78, C73 to C79, C74 to C80, C75 to C81, C76 to C82, C77 to C83, C78 to C84, C79 to C85, C80 to C86, C81 to C87, C82 to C88, C83 to C89, C84 to C90, C85 to C91, C86 to C92, C87 to C93, C88 to C94, C89 to C95, C90 to C96, H3 to H2, H7 to H4, R35 to R21, R39 to R24, R41 to R25, R44 to R28, R45 to R29, U7 to U6
Connections:
- C26 pad 1: Net-(C42-Pad1) -> Net-(C26-Pad1)
- C26 pad 2: Net-(C42-Pad2) -> Net-(C26-Pad2)
- C43 pad 1: GND -> Net-(C43-Pad1)
- C43 pad 2: V_IN -> Net-(C43-Pad2)
- C45 pad 1: GND -> V_IN
- C45 pad 2: V_IN -> GND
- C47 pad 1: GND -> V_IN
- C47 pad 2: V_IN -> GND
- C49 pad 1: V_IN -> GND
- C49 pad 2: GND -> V_IN
- C50 pad 1: /driver/HS2 -> V_IN
- C50 pad 2: Net-(C50-Pad2) -> GND
- C51 pad 1: /driver/HS2 -> GND
- C51 pad 2: Net-(C51-Pad2) -> V_IN
- C52 pad 1: VCC -> V_IN
- C53 pad 1: VCC -> V_IN
- C55 pad 1: Net-(C55-Pad1) -> /driver/HS2
- C55 pad 2: /driver/HS3 -> Net-(C55-Pad2)
- C56 pad 1: Net-(C56-Pad1) -> VCC
- C56 pad 2: Net-(C56-Pad2) -> GND
- C57 pad 1: Net-(C57-Pad1) -> VCC
- C57 pad 2: Net-(C57-Pad2) -> GND
- C60 pad 1: GND -> Net-(C60-Pad1)
- C60 pad 2: V_IN -> Net-(C60-Pad2)
- C62 pad 1: GND -> V_IN
- C62 pad 2: V_IN -> GND
- C65 pad 1: /driver/HS3 -> V_IN
- C65 pad 2: Net-(C65-Pad2) -> GND
- C66 pad 1: /driver/HS3 -> GND
- C66 pad 2: Net-(C66-Pad2) -> V_IN
- NT3 pad 1: Net-(C42-Pad2) -> Net-(C44-Pad2)
- NT3 pad 2: Net-(C41-Pad2) -> Net-(C43-Pad2)
- NT4 pad 1: Net-(C42-Pad1) -> Net-(C44-Pad1)
- NT5 pad 1: Net-(C57-Pad2) -> Net-(C61-Pad2)
- NT5 pad 2: Net-(C56-Pad2) -> Net-(C60-Pad2)
- NT6 pad 1: Net-(C57-Pad1) -> Net-(C61-Pad1)
- Q3 pad 1: Net-(C24-Pad1) -> Net-(C42-Pad1)
- Q3 pad 3: /driver/HS1 -> /driver/HS2
- Q4 pad 1: Net-(C25-Pad1) -> Net-(C43-Pad1)
- Q4 pad 2: /driver/HS1 -> /driver/HS2
- Q4 pad 3: Net-(C25-Pad2) -> Net-(C43-Pad2)
- Q5 pad 1: Net-(C40-Pad1) -> Net-(C59-Pad1)
- Q5 pad 3: /driver/HS2 -> /driver/HS3
- Q6 pad 1: Net-(C41-Pad1) -> Net-(C60-Pad1)
- Q6 pad 2: /driver/HS2 -> /driver/HS3
- Q6 pad 3: Net-(C41-Pad2) -> Net-(C60-Pad2)
- R21 pad 2: /mcu/CURRENT_2 -> /mcu/CURRENT_1
- R28 pad 1: Net-(C42-Pad2) -> Net-(C26-Pad2)
- R29 pad 1: Net-(C42-Pad1) -> Net-(C26-Pad1)
- R37 pad 2: Net-(C40-Pad1) -> Net-(C42-Pad1)
- R38 pad 2: Net-(C41-Pad1) -> Net-(C43-Pad1)
- R42 pad 2: Net-(C40-Pad1) -> Net-(C42-Pad1)
- R43 pad 1: Net-(C41-Pad2) -> Net-(C43-Pad2)
- R43 pad 2: Net-(C41-Pad1) -> Net-(C43-Pad1)
- R46 pad 1: Net-(C41-Pad2) -> Net-(C43-Pad2)
- R47 pad 1: Net-(C50-Pad2) -> Net-(C54-Pad2)
- R48 pad 1: Net-(C51-Pad2) -> Net-(C55-Pad2)
- R49 pad 1: Net-(C50-Pad2) -> Net-(C54-Pad2)
- R50 pad 1: Net-(C51-Pad2) -> Net-(C55-Pad2)
- R52 pad 2: Net-(C55-Pad1) -> Net-(C59-Pad1)
- R53 pad 2: Net-(C56-Pad1) -> Net-(C60-Pad1)
- R56 pad 2: Net-(C55-Pad1) -> Net-(C59-Pad1)
- R57 pad 1: Net-(C56-Pad2) -> Net-(C60-Pad2)
- R57 pad 2: Net-(C56-Pad1) -> Net-(C60-Pad1)
- R58 pad 1: Net-(C57-Pad2) -> Net-(C61-Pad2)
- R59 pad 1: Net-(C57-Pad1) -> Net-(C61-Pad1)
- R60 pad 1: Net-(C56-Pad2) -> Net-(C60-Pad2)
- R61 pad 1: Net-(C65-Pad2) -> Net-(C71-Pad2)
- R62 pad 1: Net-(C66-Pad2) -> Net-(C72-Pad2)
- R63 pad 1: Net-(C65-Pad2) -> Net-(C71-Pad2)
- R64 pad 1: Net-(C66-Pad2) -> Net-(C72-Pad2)
Routing:
- net +12V: track 255.7 -> 295.1 mm, vias 8 -> 4
- net Net-(C41-Pad1): track 26.1 -> 0.00 mm
- net Net-(C61-Pad1): track 0.00 -> 25.9 mm, vias 0 -> 1
- net Net-(C61-Pad2): track 0.00 -> 25.6 mm
- net Net-(C44-Pad2): track 0.00 -> 25.4 mm, vias 0 -> 1
- net Net-(C44-Pad1): track 0.00 -> 25.0 mm, vias 0 -> 1
- net Net-(C40-Pad1): track 21.5 -> 0.00 mm
- net Net-(C55-Pad1): track 21.4 -> 0.00 mm
- net Net-(C56-Pad1): track 20.7 -> 0.00 mm
- net Net-(C57-Pad2): track 20.0 -> 0.00 mm, vias 1 -> 0
- net Net-(C42-Pad2): track 19.4 -> 0.00 mm, vias 1 -> 0
- net Net-(C57-Pad1): track 17.9 -> 0.00 mm, vias 1 -> 0
- net /driver/HS3: track 23.8 -> 9.21 mm
- net /driver/HS1: track 23.8 -> 9.78 mm
- net /driver/HO2: track 20.1 -> 6.19 mm
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- added copper zone on F.Cu, net /driver/HS1
- added copper zone on F.Cu, net /driver/HS2
- added copper zone on F.Cu, net /driver/HS3
- added copper zone on F.Cu, net V_IN
Other:
- board size 68.4 x 79 mm -> 60.7 x 89.9 mm
- board text added: "++++++"
- board text added: "------"
- board text added: "2023 jens overby github.com/nordstream3/FOC"
- board text added: "UFO.CIA"
- board text removed: "A"
- board text removed: "B"
- board text removed: "C"
- board text removed: "NEG"
- board text removed: "POS"
- board text removed: "WATT'EVER"
- board text removed: "github.com/nordstream3/FOC"

Commit message: Add files via upload
Parts:
- removed the C11 at (113.0, 123.2)
- removed the R70 at (97.6, 139.1)
- added C3: 100n, Resistor_SMD:R_0603_1608Metric, F.Cu at (78.8, 144.0)
- added J1: Conn_01x06, Connector_JST:JST_PH_B6B-PH-K_1x06_P2.00mm_Vertical, F.Cu at (89.5, 147.9)
- added J2: Conn_01x08, Connector_JST:JST_PH_B8B-PH-K_1x08_P2.00mm_Vertical, F.Cu at (67.1, 138.4)
- added J3: NRF wireless, Connector_PinSocket_2.54mm:PinSocket_2x04_P2.54mm_Vertical, F.Cu at (102.3, 132.9)
- added R1: 2k2, Resistor_SMD:R_0603_1608Metric, F.Cu at (81.8, 144.0)
- added R2: 2k2, Resistor_SMD:R_0603_1608Metric, F.Cu at (84.7, 144.0)
- added R3: 2k2, Resistor_SMD:R_0603_1608Metric, F.Cu at (87.6, 144.0)
- added R5: 10k, Resistor_SMD:R_0603_1608Metric, F.Cu at (76.5, 143.2)
- added R74: 20k, Resistor_SMD:R_0603_1608Metric, F.Cu at (96.2, 139.1)
- added SW1: SW_DPDT_x2, Jumper:SolderJumper-3_P1.3mm_Bridged2Bar12_Pad1.0x1.5mm, F.Cu at (76.5, 146.6)
- Q1: value NCEP60T20 -> CSD19536KCS
- moved R75 10.0 mm to (110.9, 140.4), turned to 180 degrees
- moved P1 9.74 mm to (98.9, 148.1)
- moved U12 8.20 mm to (69.0, 117.2)
- moved C92 8.09 mm to (68.4, 112.2), turned to 180 degrees
- moved R15 7.33 mm to (114.8, 125.0)
- moved C83 7.21 mm to (93.5, 145.3), turned to 180 degrees
- moved D12 6.35 mm to (107.9, 140.4), turned to 180 degrees
- moved H2 5.40 mm to (112.6, 116.9)
- moved H1 4.80 mm to (74.8, 117.0)
- moved U10 4.26 mm to (108.1, 144.0)
- moved R6 2.66 mm to (74.1, 135.5)
- moved R4 2.63 mm to (74.1, 134.0)
- moved C1 2.53 mm to (73.7, 129.2)
- moved C2 2.53 mm to (71.5, 129.9)
- moved U1 2.53 mm to (74.1, 131.7)
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- renumbered C9 to C10, C10 to C11, C3 to C4, C4 to C5, C5 to C6, C6 to C7, C7 to C8, C8 to C9, J1 to J4, J2 to J5, R6 to R10, R7 to R11, R8 to R12, R9 to R13, R10 to R14, R11 to R15, R12 to R16, R13 to R17, R14 to R18, R15 to R19, R16 to R20, R17 to R21, R18 to R22, R19 to R23, R20 to R24, R21 to R25, R22 to R26, R23 to R27, R24 to R28, R25 to R29, R26 to R30, R27 to R31, R28 to R32, R29 to R33, R30 to R34, R31 to R35, R32 to R36, R33 to R37, R34 to R38, R35 to R39, R1 to R4, R36 to R40, R37 to R41, R38 to R42, R39 to R43, R40 to R44, R41 to R45, R42 to R46, R43 to R47, R44 to R48, R45 to R49, R46 to R50, R47 to R51, R48 to R52, R49 to R53, R50 to R54, R51 to R55, R52 to R56, R53 to R57, R54 to R58, R55 to R59, R2 to R6, R56 to R60, R57 to R61, R58 to R62, R59 to R63, R60 to R64, R61 to R65, R62 to R66, R63 to R67, R64 to R68, R65 to R69, R3 to R7, R66 to R70, R67 to R71, R68 to R72, R69 to R73, R71 to R75, R4 to R8, R5 to R9
Connections:
- U11 pad 20: unconnected-(U11-Pad20) -> /mcu/RX_SDA_NSS
- U11 pad 21: unconnected-(U11-Pad21) -> /mcu/SCK_ADC_EXT
- U11 pad 22: unconnected-(U11-Pad22) -> /mcu/MISO_ADC_EXT2
- U11 pad 23: unconnected-(U11-Pad23) -> /mcu/TX_SCL_MOSI
- U11 pad 25: unconnected-(U11-Pad25) -> /mcu/ADC_15
- U11 pad 51: unconnected-(U11-Pad51) -> /mcu/SERVO
- U11 pad 54: unconnected-(U11-Pad54) -> /mcu/NRF_MISO
- U11 pad 55: unconnected-(U11-Pad55) -> /mcu/NRF_MOSI
- U11 pad 56: unconnected-(U11-Pad56) -> /mcu/NRF_SCK
- U11 pad 58: /mcu/SERVO -> /mcu/LED_RED
- U11 pad 59: /mcu/LED_RED -> /mcu/NRF_CSN
Routing:
- net VCC: track 199.7 -> 266.9 mm
- net GND: track 179.0 -> 133.7 mm, vias 878 -> 964
- net +5V: track 57.8 -> 95.4 mm, vias 0 -> 2
- net /mcu/RX_SDA_NSS: track 0.00 -> 35.3 mm
- net /mcu/SCK_ADC_EXT: track 0.00 -> 29.2 mm
- net /mcu/ADC_15: track 0.00 -> 25.1 mm, vias 0 -> 2
- net Net-(J1-Pad6): track 0.00 -> 23.7 mm, vias 0 -> 2
- net /mcu/MISO_ADC_EXT2: track 0.00 -> 23.3 mm
- net /mcu/TX_SCL_MOSI: track 0.00 -> 22.1 mm
- net /mcu/TEMP_MOTOR: track 0.00 -> 20.2 mm, vias 0 -> 2
- net /driver/H1: track 59.2 -> 76.3 mm
- net /mcu/USB_D+: track 27.2 -> 42.8 mm
- net /mcu/USB_D-: track 27.3 -> 42.8 mm
- net V_IN: track 88.2 -> 74.1 mm
- net /mcu/NRF_CSN: track 0.00 -> 11.0 mm
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Other:
- board text added: "FOC"
- board text added: "IMU"
- board text added: "KING"
- board text added: "NRF"
- board text added: "wireless"
- board text removed: "UFO.CIA"
