File: source/foc.kicad_pcb (KiCad board)
At the start: 2 copper layers, 60.7 x 89.9 mm, 224 parts, among them J1 Conn_01x06, J2 Conn_01x08, J3 NRF wireless, J4 Conn_01x04_Male, J5 TYPE-C-31-M-12, P1 SWD, Q1 CSD19536KCS, Q2 CSD19536KCS, Q3 CSD19536KCS, Q4 CSD19536KCS, Q5 CSD19536KCS, Q6 CSD19536KCS, SW1 SW_DPDT_x2, U1 BMI160, U10 HT7550, U11 STM32F405RGT6, U12 AMS1117-3.3, U2 IRS21867S, U3 IRS21867S, U4 IRS21867S, U5 TX4130L/PW2902, U6 MS8311, U7 MS8311, U8 MS8311, U9 TJA1050T/CM,118, Y1 8MHz Crystal Resonator, X5032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

Commit message: Add files via upload
Parts:
- removed the C12 at (106.7, 105.4)
- removed the C42 at (85.7, 95.7)
- removed the C43 at (92.1, 95.7)
- removed the C59 at (106.1, 95.7)
- removed the C60 at (112.5, 95.7)
- removed the C79 at (111.7, 143.9)
- removed the C92 at (68.4, 112.2)
- removed the C96 at (77.0, 123.5)
- removed the D4 at (93.8, 102.8)
- removed the D7 at (106.8, 100.3)
- removed the J3 at (102.3, 132.9)
- removed the R19 at (109.3, 95.7)
- removed the R41 at (84.7, 99.5)
- removed the R42 at (93.6, 99.6)
- removed the R56 at (105.1, 99.5)
- removed the R57 at (114.0, 99.6)
- removed the R60 at (106.1, 97.2)
- removed the R9 at (68.6, 95.7)
- removed the U10 at (108.1, 144.0)
- removed the U12 at (69.0, 117.2)
- removed the U4 at (110.5, 101.8)
- added C15: 15n, Capacitor_SMD:C_0603_1608Metric, F.Cu at (161.7, 131.2)
- added C17: 1n, Capacitor_SMD:C_0603_1608Metric, F.Cu at (161.7, 133.7)
- added C18: 1u, Capacitor_SMD:C_0603_1608Metric, F.Cu at (88.9, 97.2)
- added C19: 100u, Capacitor_Tantalum_SMD:CP_EIA-3528-21_Kemet-B, F.Cu at (113.4, 144.6)
- added C20: 15n, Capacitor_SMD:C_0603_1608Metric, F.Cu at (157.4, 135.0)
- added C21: 100u@6.3V, Capacitor_SMD:C_1206_3216Metric, F.Cu at (120.8, 145.0)
- added C22: 1n, Capacitor_SMD:C_0603_1608Metric, F.Cu at (157.2, 138.8)
- added C23: 10u, Capacitor_Tantalum_SMD:CP_EIA-3216-10_Kemet-I, F.Cu at (106.6, 105.9)
- added C24: 2.2u, Capacitor_SMD:C_0603_1608Metric, F.Cu at (108.4, 106.8)
- added C27: 1u, Capacitor_SMD:C_0603_1608Metric, F.Cu at (109.2, 97.2)
- added C3: 100n, Resistor_SMD:R_0603_1608Metric, F.Cu at (78.3, 138.6)
- added C53: 2.2nF, Capacitor_SMD:C_0603_1608Metric, F.Cu at (88.9, 94.2)
- added C54: 2.2nF, Capacitor_SMD:C_0603_1608Metric, F.Cu at (94.5, 95.6)
- added C6: 100n, Capacitor_SMD:C_0603_1608Metric, F.Cu at (66.7, 111.3)
- added C70: 2.2nF, Capacitor_SMD:C_0603_1608Metric, F.Cu at (109.2, 94.2)
- added C71: 2.2nF, Capacitor_SMD:C_0603_1608Metric, F.Cu at (114.8, 95.6)
- added CYA0650-68UH1: 68uH, Custom:L_6.6x7.2_H5.0_CYA0650_68UH, F.Cu at (120.0, 140.0)
- added D10: 1N5819WS, Diode_SMD:D_SOD-323, F.Cu at (86.4, 98.1)
- added D11: 1N5819WS, Diode_SMD:D_SOD-323, F.Cu at (95.2, 98.7)
- added D12: 1N5819WS, Diode_SMD:D_SOD-323, F.Cu at (106.8, 98.1)
- added D13: 1N5819WS, Diode_SMD:D_SOD-323, F.Cu at (115.5, 98.6)
- added D6: 1N4148WS, Diode_SMD:D_SOD-323, F.Cu at (106.8, 101.3)
- added D9: 1N5819WS, Diode_SMD:D_SOD-323, F.Cu at (74.9, 98.7)
- added J1: Conn_01x03, Connector_JST:JST_PH_B3B-PH-K_1x03_P2.00mm_Vertical, F.Cu at (67.5, 148.4)
- added J4: NRF wireless, Connector_PinSocket_2.54mm:PinSocket_2x04_P2.54mm_Vertical, B.Cu at (101.5, 130.1)
- added Q1: MMBT5401, Package_TO_SOT_SMD:SOT-23, F.Cu at (65.4, 94.6)
- added Q10: MMBT5401, Package_TO_SOT_SMD:SOT-23, F.Cu at (112.4, 96.0)
- added Q2: MMBT5401, Package_TO_SOT_SMD:SOT-23, F.Cu at (71.8, 96.0)
- added Q5: MMBT5401, Package_TO_SOT_SMD:SOT-23, F.Cu at (85.7, 94.6)
- added Q6: MMBT5401, Package_TO_SOT_SMD:SOT-23, F.Cu at (92.1, 96.0)
- added Q9: MMBT5401, Package_TO_SOT_SMD:SOT-23, F.Cu at (106.1, 94.6)
- added R10: 1k, Resistor_SMD:R_0603_1608Metric, F.Cu at (165.7, 131.2)
- added R11: 1k, Resistor_SMD:R_0603_1608Metric, F.Cu at (153.2, 138.8)
- added R27: 2k2, Resistor_SMD:R_0603_1608Metric, F.Cu at (64.4, 98.0)
- added R28: 2k2, Resistor_SMD:R_0603_1608Metric, F.Cu at (73.2, 99.4)
- added R4: 100R, Resistor_SMD:R_0603_1608Metric, F.Cu at (75.3, 138.6)
- added R44: 2k2, Resistor_SMD:R_0603_1608Metric, F.Cu at (84.7, 98.0)
- added R45: 2k2, Resistor_SMD:R_0603_1608Metric, F.Cu at (93.5, 99.4)
- added R53: 4.7k @ 75v, Resistor_SMD:R_0603_1608Metric, F.Cu at (88.9, 95.7)
- added R54: 4.7k @ 75v, Resistor_SMD:R_0603_1608Metric, F.Cu at (96.0, 95.6)
- added R62: 2k2, Resistor_SMD:R_0603_1608Metric, F.Cu at (113.9, 99.4)
- added R63: 4.7R, Resistor_SMD:R_0603_1608Metric, F.Cu at (105.1, 101.2)
- added R64: 4.7R, Resistor_SMD:R_0603_1608Metric, F.Cu at (114.6, 101.6)
- added R69: 4.7k @ 75v, Resistor_SMD:R_0603_1608Metric, F.Cu at (109.2, 95.7)
- added R70: 4.7k @ 75v, Resistor_SMD:R_0603_1608Metric, F.Cu at (116.3, 95.6)
- added U2: AMS1117-3.3, Package_TO_SOT_SMD:SOT-223-3_TabPin2, F.Cu at (69.0, 117.2)
- added U5: MC74VHC1G66, Package_TO_SOT_SMD:SOT-353_SC-70-5, F.Cu at (157.5, 131.8)
- added U6: XL1509-5.0E1, Package_SO:SOP-8_3.9x4.9mm_P1.27mm, F.Cu at (113.3, 139.2)
- added U7: EG3112, Package_SO:SOIC-8_3.9x4.9mm_P1.27mm, F.Cu at (90.1, 101.6)
- added U8: MC74VHC1G66, Package_TO_SOT_SMD:SOT-353_SC-70-5, F.Cu at (153.3, 131.8)
- added U9: EG3112, Package_SO:SOIC-8_3.9x4.9mm_P1.27mm, F.Cu at (110.4, 101.6)
- C10: value 2.2u -> 1n
- C11: value 1u -> 100u@6.3V; footprint Capacitor_SMD:C_0603_1608Metric -> Capacitor_SMD:C_1206_3216Metric
- C14: value 2.2u -> 10u; footprint Capacitor_SMD:C_0603_1608Metric -> Capacitor_Tantalum_SMD:CP_EIA-3216-10_Kemet-I
- C16: value 1u -> 2.2u
- C9: value 10u -> 15n; footprint Capacitor_Tantalum_SMD:CP_EIA-3216-10_Kemet-I -> Capacitor_SMD:C_0603_1608Metric
- D2: value 1N4148WS -> 1N5819
- D8: value 1N4148WS -> 1N5819WS
- R14: value 2R -> 1k
- R46, R47: value 4.7k @ 75v -> 4.7R
- R61: value 4.7k @ 75v -> 2k2
- R76: renamed from R69; value 100Ω -> 100R
- R77: renamed from R70; value 100Ω -> 100R
- R80: renamed from R73; value 20k -> 10k
- R81: renamed from R74; value 20k -> 10k
- U3: value IRS21867S -> MC74VHC1G66; footprint Package_SO:SOIC-8_3.9x4.9mm_P1.27mm -> Package_TO_SOT_SMD:SOT-353_SC-70-5
- U4: renamed from U2; value IRS21867S -> EG3112
- moved C9 81.1 mm to (161.4, 136.2), turned to 0 degrees
- moved R14 78.8 mm to (153.2, 141.4), turned to 0 degrees
- moved C10 77.1 mm to (157.2, 141.4), turned to 0 degrees
- moved U3 71.7 mm to (153.3, 135.7), turned to 0 degrees
- moved D2 54.8 mm to (117.6, 135.3), turned to 180 degrees
- moved R82 50.4 mm to (69.7, 111.3), turned to 90 degrees
- moved D16 49.2 mm to (68.2, 111.3), turned to -90 degrees
- moved D8 48.3 mm to (66.1, 98.1)
- moved C11 30.2 mm to (75.2, 124.1), turned to 90 degrees
- moved R79 27.2 mm to (98.5, 144.8), turned to -90 degrees
- moved J6 23.5 mm to (92.6, 146.5)
- moved C16 23.3 mm to (88.1, 106.8), turned to -90 degrees
- moved C14 22.2 mm to (86.3, 106.0)
- moved R78 20.2 mm to (86.8, 144.0), turned to -90 degrees
- moved R77 16.4 mm to (108.1, 137.3), turned to 0 degrees
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- renumbered C90 to C100, C91 to C101, C93 to C102, C94 to C103, C95 to C104, C7 to C12, C6 to C13, C13 to C25, C15 to C26, C17 to C28, C18 to C29, C19 to C30, C20 to C31, C21 to C32, C22 to C33, C23 to C34, C24 to C35, C25 to C36, C26 to C37, C27 to C38, C28 to C39, C3 to C4, C29 to C40, C30 to C41, C31 to C42, C32 to C43, C33 to C44, C34 to C45, C35 to C46, C36 to C47, C37 to C48, C38 to C49, C4 to C5, C39 to C50, C40 to C51, C41 to C52, C44 to C55, C45 to C56, C46 to C57, C47 to C58, C48 to C59, C49 to C60, C50 to C61, C51 to C62, C52 to C63, C53 to C64, C54 to C65, C55 to C66, C56 to C67, C57 to C68, C58 to C69, C5 to C7, C61 to C72, C62 to C73, C63 to C74, C64 to C75, C65 to C76, C66 to C77, C67 to C78, C68 to C79, C69 to C80, C70 to C81, C71 to C82, C72 to C83, C73 to C84, C74 to C85, C75 to C86, C76 to C87, C77 to C88, C78 to C89, C80 to C90, C81 to C91, C82 to C92, C83 to C93, C84 to C94, C85 to C95, C86 to C96, C87 to C97, C88 to C98, C89 to C99, CYA0650-68UH1 to CYA0650-68UH2, D10 to D14, D11 to D15, D12 to D16, D5 to D4, D6 to D5, D9 to D7, J1 to J2, J2 to J3, J4 to J5, J5 to J6, Q5 to Q11, Q6 to Q12, Q1 to Q3, Q2 to Q4, Q3 to Q7, Q4 to Q8, R20 to R19, R21 to R20, R22 to R21, R23 to R22, R24 to R23, R10 to R24, R11 to R25, R25 to R26, R26 to R29, R27 to R30, R28 to R31, R29 to R32, R32 to R33, R33 to R34, R30 to R35, R31 to R36, R34 to R37, R35 to R38, R36 to R39, R37 to R40, R38 to R41, R39 to R42, R40 to R43, R43 to R48, R44 to R49, R4 to R5, R45 to R50, R48 to R51, R49 to R52, R50 to R55, R51 to R56, R52 to R57, R53 to R58, R54 to R59, R5 to R6, R55 to R60, R58 to R65, R59 to R66, R62 to R67, R63 to R68, R6 to R7, R64 to R71, R65 to R72, R66 to R73, R67 to R74, R68 to R75, R71 to R78, R72 to R79, R7 to R8, R75 to R82, R8 to R9, U5 to U10, U6 to U11, U7 to U12, U8 to U13, U9 to U14, U11 to U15
Connections:
- C10 pad 1: +12V -> /driver/CURR_A
- C11 pad 1: Net-(C11-Pad1) -> VCC
- C11 pad 2: Net-(C11-Pad2) -> GND
- C12 pad 2: Net-(C7-Pad2) -> /driver/HS1
- C14 pad 2: GND -> Net-(C14-Pad2)
- C16 pad 1: Net-(C16-Pad1) -> +12V
- C16 pad 2: Net-(C16-Pad2) -> Net-(C14-Pad2)
- C34 pad 2: /mcu/CURRENT_1 -> /driver/C_A
- C35 pad 1: Net-(C24-Pad1) -> Net-(C35-Pad1)
- C36 pad 1: Net-(C25-Pad1) -> Net-(C36-Pad1)
- C51 pad 2: /mcu/CURRENT_2 -> /driver/C_B
- C69 pad 2: /mcu/CURRENT_3 -> /driver/C_C
- C9 pad 1: +12V -> Net-(C9-Pad1)
- D2 pad 1: Net-(C7-Pad2) -> Net-(CYA0650-68UH1-Pad1)
- D3 pad 1: Net-(C11-Pad1) -> Net-(C18-Pad1)
- D8 pad 1: Net-(C16-Pad2) -> Net-(C35-Pad1)
- D8 pad 2: GND -> Net-(D8-Pad2)
- J6 pad A4B9: +5V -> unconnected-(J6-PadA4B9)
- J6 pad B4A9: +5V -> unconnected-(J6-PadB4A9)
- NT3 pad 2: Net-(C43-Pad2) -> Net-(C54-Pad2)
- NT5 pad 2: Net-(C60-Pad2) -> Net-(C71-Pad2)
- P1 pad 1: /mcu/NRST -> VCC
- P1 pad 2: /mcu/SWDIO -> /mcu/SWCLK
- P1 pad 4: /mcu/SWCLK -> /mcu/SWDIO
- P1 pad 5: VCC -> /mcu/NRST
- Q12 pad 1: Net-(C60-Pad1) -> Net-(C71-Pad1)
- Q12 pad 3: Net-(C60-Pad2) -> Net-(C71-Pad2)
- Q3 pad 1: Net-(C24-Pad1) -> Net-(C35-Pad1)
- Q4 pad 1: Net-(C25-Pad1) -> Net-(C36-Pad1)
- Q7 pad 1: Net-(C42-Pad1) -> Net-(C53-Pad1)
- Q8 pad 1: Net-(C43-Pad1) -> Net-(C54-Pad1)
- Q8 pad 3: Net-(C43-Pad2) -> Net-(C54-Pad2)
- R14 pad 1: Net-(C11-Pad2) -> /driver/CURR_C
- R14 pad 2: /driver/HS2 -> /driver/C_C
- R26 pad 2: /mcu/CURRENT_1 -> /driver/C_A
- R29 pad 2: Net-(C24-Pad1) -> Net-(D8-Pad2)
- R30 pad 2: Net-(C25-Pad1) -> Net-(D9-Pad2)
- R35 pad 2: Net-(C24-Pad1) -> Net-(C35-Pad1)
- R36 pad 2: Net-(C25-Pad1) -> Net-(C36-Pad1)
- R42 pad 2: /mcu/CURRENT_2 -> /driver/C_B
- R46 pad 1: /driver/HS2 -> /driver/HO2
- R46 pad 2: Net-(C42-Pad1) -> Net-(D10-Pad2)
- R47 pad 1: Net-(C43-Pad2) -> /driver/LO2
- R47 pad 2: Net-(C43-Pad1) -> Net-(D11-Pad2)
- R55 pad 1: Net-(C43-Pad2) -> Net-(C54-Pad2)
- R60 pad 2: /mcu/CURRENT_3 -> /driver/C_C
- R61 pad 1: Net-(C60-Pad2) -> Net-(Q9-Pad1)
- R61 pad 2: Net-(C60-Pad1) -> Net-(D12-Pad2)
- R71 pad 1: Net-(C60-Pad2) -> Net-(C71-Pad2)
- U15 pad 11: /mcu/CURRENT_2 -> /driver/CURR_B
- U15 pad 16: /mcu/CURRENT_1 -> /driver/CURR_A
- U15 pad 2: unconnected-(U11-Pad2) -> /driver/CURR_FILTER
- U15 pad 27: unconnected-(U11-Pad27) -> /mcu/SERVO
- U15 pad 29: unconnected-(U11-Pad29) -> /mcu/TX_SCL_MOSI
- U15 pad 30: unconnected-(U11-Pad30) -> /mcu/RX_SDA_NSS
- U15 pad 51: /mcu/SERVO -> unconnected-(U15-Pad51)
- U15 pad 8: /mcu/CURRENT_3 -> /driver/CURR_C
- U3 pad 1: +12V -> /driver/CURR_A
- U3 pad 2: /driver/H2 -> Net-(C9-Pad1)
- U3 pad 3: /driver/L2 -> GND
- U3 pad 4: GND -> /driver/CURR_FILTER
- U3 pad 5: /driver/LO2 -> VCC
- U4 pad 6: Net-(C7-Pad2) -> /driver/HS1
Routing:
- net GND: track 133.7 -> 71.8 mm, vias 964 -> 912
- net /mcu/CURRENT_3: track 42.1 -> 0.00 mm
- net /driver/C_C: track 0.00 -> 37.8 mm
- net /mcu/USB_D+: track 42.8 -> 8.33 mm
- net /mcu/USB_D-: track 42.8 -> 8.98 mm
- net +5V: track 95.4 -> 128.1 mm, vias 2 -> 3
- net +12V: track 292.7 -> 264.3 mm
- net /mcu/CURRENT_2: track 26.7 -> 0.00 mm
- net /driver/C_B: track 0.00 -> 24.9 mm
- net /mcu/CURRENT_1: track 20.2 -> 0.00 mm
- net /driver/C_A: track 0.00 -> 16.1 mm
- net Net-(C89-Pad1): track 4.64 -> 20.4 mm
- net Net-(J1-Pad1): track 0.00 -> 15.3 mm, vias 0 -> 2
- net Net-(C88-Pad1): track 4.97 -> 18.7 mm
- net /mcu/SERVO: track 0.00 -> 13.6 mm
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Other:
- board text added: "+5V"
- board text added: "{"

Commit message: Add files via upload
Parts:
- removed the C10 at (157.2, 141.4)
- removed the C18 at (88.9, 97.2)
- removed the C22 at (157.2, 138.8)
- removed the C23 at (106.6, 105.9)
- removed the C27 at (109.2, 97.2)
- removed the C46 at (70.8, 69.5)
- removed the C72 at (117.8, 103.7)
- removed the R14 at (153.2, 141.4)
- removed the R16 at (119.4, 90.2)
- removed the R17 at (121.6, 89.5)
- removed the R24 at (84.3, 89.9)
- removed the R25 at (84.3, 92.9)
- removed the R73 at (118.6, 86.5)
- removed the R74 at (111.6, 87.6)
- removed the R75 at (120.1, 86.5)
- added C13: 10u, Capacitor_Tantalum_SMD:CP_EIA-3216-10_Kemet-I, F.Cu at (85.2, 105.9)
- added C21: 2.2u, Capacitor_SMD:C_0603_1608Metric, F.Cu at (107.9, 106.8)
- added C41: 100n 100V, Capacitor_SMD:C_0805_2012Metric, F.Cu at (64.0, 78.0)
- added C43: 100n 100V, Capacitor_SMD:C_0805_2012Metric, F.Cu at (64.0, 76.0)
- added C45: 100n 100V, Capacitor_SMD:C_0805_2012Metric, F.Cu at (63.9, 85.9)
- added C84: 100n 100V, Capacitor_SMD:C_0805_2012Metric, F.Cu at (106.1, 75.9)
- added C85: 100n 100V, Capacitor_SMD:C_0805_2012Metric, F.Cu at (116.2, 74.0)
- added C86: 100n 100V, Capacitor_SMD:C_0805_2012Metric, F.Cu at (106.1, 85.9)
- added C87: 4.7n, Capacitor_SMD:C_0603_1608Metric, F.Cu at (116.7, 85.0)
- added C88: 4.7n, Capacitor_SMD:C_0603_1608Metric, F.Cu at (118.1, 86.5)
- added H8: MountingHole, MountingHole:MountingHole_4.3mm_M4_Pad_TopOnly, B.Cu at (108.3, 91.4)
- added R21: 56k @ 75V, Resistor_SMD:R_0603_1608Metric, F.Cu at (82.7, 87.1)
- added R22: 2k, Resistor_SMD:R_0603_1608Metric, F.Cu at (82.7, 90.0)
- added R39: 30k, Resistor_SMD:R_0603_1608Metric, F.Cu at (99.1, 112.6)
- added R40: NTC 10k, Resistor_SMD:R_0603_1608Metric, F.Cu at (70.2, 96.6)
- added R41: 2k2, Resistor_SMD:R_0603_1608Metric, F.Cu at (95.1, 93.8)
- C14: value 10u -> 100n; footprint Capacitor_Tantalum_SMD:CP_EIA-3216-10_Kemet-I -> Capacitor_SMD:C_0603_1608Metric
- C15: value 15n -> 2.2u
- C16, C24: value 2.2u -> 1u
- C17: value 1n -> 100n
- C20: value 15n -> 10u; footprint Capacitor_SMD:C_0603_1608Metric -> Capacitor_Tantalum_SMD:CP_EIA-3216-10_Kemet-I
- C42, C44, C60, C62, C77, C79: value 10u @ 100V -> 100n 100V; footprint Capacitor_SMD:C_2220_5650Metric -> Capacitor_SMD:C_0805_2012Metric
- C64, C81: value 470u 80V -> 100n 100V; footprint Capacitor_THT:CP_Radial_D10.0mm_P5.00mm -> Capacitor_SMD:C_0805_2012Metric
- C65, C66, C82, C83: value 4.7n -> 100n 100V; footprint Capacitor_SMD:C_0603_1608Metric -> Capacitor_SMD:C_0805_2012Metric
- C67: value 2.2u -> 4.7n
- C68: value 100n -> 4.7n
- C70: value 2.2nF -> 2.2u
- C71: value 2.2nF -> 100n
- C73, C74: value 100n 100V -> 2.2nF; footprint Capacitor_SMD:C_0805_2012Metric -> Capacitor_SMD:C_0603_1608Metric
- C75: value 100n 100V -> 100p; footprint Capacitor_SMD:C_0805_2012Metric -> Capacitor_SMD:C_0603_1608Metric
- C9: value 15n -> 100n
- H6, H7: value MountingHole_Pad -> MountingHole; footprint MountingHole:MountingHole_4mm_Pad_TopOnly -> MountingHole:MountingHole_4.3mm_M4_Pad_TopOnly; moved to B.Cu
- J4: moved to F.Cu
- R10: value 1k -> 56k @ 75V
- R11: value 1k -> 2k
- R42: value 30k -> 2k2
- R43: value NTC 10k -> 4.7R
- R44, R61: value 2k2 -> 4.7R
- R45, R62: value 2k2 -> 30k
- R46: value 4.7R -> 10k
- R47, R63: value 4.7R -> 62k
- R48, R65: value 30k -> 1k
- R49: value 10k -> 1k
- R50, R66: value 62k -> 4.7k @ 75v
- R51, R67: value 1k -> 4.7k @ 75v
- R52, R68: value 1k -> ASR-M-3-0.25F 0.25mR; footprint Resistor_SMD:R_0603_1608Metric -> Resistor_SMD:R_2512_6332Metric; moved to B.Cu
- R53, R54, R69, R70: value 4.7k @ 75v -> 10R
- R55, R71: value ASR-M-3-0.25F 0.25mR -> 10R; footprint Resistor_SMD:R_2512_6332Metric -> Resistor_SMD:R_0603_1608Metric; moved to F.Cu
- R57: value 10R -> 30k
- R58, R59: value 10R -> 2k2
- R60: value 30k -> 4.7R
- R64: value 4.7R -> 1k
- moved C9 81.2 mm to (81.5, 121.9), turned to -90 degrees
- moved C15 78.5 mm to (87.0, 106.8), turned to -90 degrees
- moved U3 72.6 mm to (81.5, 125.0), turned to -90 degrees
- moved U5 72.1 mm to (86.3, 120.4), turned to 180 degrees
- moved R10 71.2 mm to (101.3, 100.6), turned to 90 degrees
- moved C17 63.7 mm to (98.6, 125.0)
- moved R11 62.7 mm to (101.3, 103.6), turned to -90 degrees
- moved C20 58.9 mm to (106.1, 105.9), turned to -90 degrees
- moved U8 54.6 mm to (98.9, 126.9), turned to 180 degrees
- moved H6 44.3 mm to (66.2, 91.4), turned to 180 degrees
- moved R57 31.3 mm to (117.4, 111.3), turned to 180 degrees
- moved C67 30.9 mm to (95.7, 85.0), turned to 0 degrees
- moved C68 29.8 mm to (97.2, 86.5), turned to 0 degrees
- moved H7 27.4 mm to (87.4, 91.4), turned to 180 degrees
- moved R58 25.6 mm to (116.0, 93.8), turned to 0 degrees
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- renumbered C11 to C10, C94 to C100, C95 to C101, C96 to C102, C97 to C103, C98 to C104, C99 to C105, C100 to C106, C101 to C107, C102 to C108, C103 to C109, C12 to C11, C104 to C110, C13 to C12, C19 to C18, C21 to C19, C25 to C22, C26 to C23, C28 to C25, C29 to C26, C30 to C27, C31 to C28, C32 to C29, C33 to C30, C34 to C31, C35 to C32, C36 to C33, C37 to C34, C38 to C35, C39 to C36, C40 to C37, C41 to C38, C43 to C39, C45 to C40, C47 to C46, C48 to C47, C69 to C72, C84 to C90, C85 to C91, C86 to C92, C87 to C93, C88 to C94, C89 to C95, C90 to C96, C91 to C97, C92 to C98, C93 to C99, R15 to R14, R18 to R15, R19 to R16, R20 to R17, R21 to R18, R22 to R19, R23 to R20, R26 to R23, R27 to R24, R28 to R25, R29 to R26, R30 to R27, R31 to R28, R32 to R29, R33 to R30, R34 to R31, R35 to R32, R36 to R33, R37 to R34, R38 to R35, R39 to R36, R40 to R37, R41 to R38, R76 to R73, R77 to R74, R78 to R75, R79 to R76, R80 to R77, R81 to R78, R82 to R79
Connections:
- C14 pad 1: +12V -> /driver/SENS_2
- C15 pad 1: Net-(C15-Pad1) -> +12V
- C15 pad 2: GND -> Net-(C13-Pad2)
- C16 pad 1: +12V -> Net-(C16-Pad1)
- C16 pad 2: Net-(C14-Pad2) -> /driver/HS2
- C17 pad 1: /driver/CURR_B -> /driver/SENS_3
- C17 pad 2: GND -> Net-(C17-Pad2)
- C20 pad 1: Net-(C20-Pad1) -> +12V
- C24 pad 1: +12V -> Net-(C24-Pad1)
- C24 pad 2: GND -> /driver/HS3
- C31 pad 2: /driver/C_A -> /mcu/CURRENT_1
- C42 pad 1: GND -> V_IN
- C42 pad 2: V_IN -> GND
- C44 pad 1: GND -> V_IN
- C44 pad 2: V_IN -> GND
- C51 pad 2: /driver/C_B -> /mcu/CURRENT_2
- C60 pad 1: GND -> V_IN
- C60 pad 2: V_IN -> GND
- C62 pad 1: GND -> V_IN
- C62 pad 2: V_IN -> GND
- C65 pad 1: /driver/HS2 -> V_IN
- C65 pad 2: Net-(C65-Pad2) -> GND
- C66 pad 1: /driver/HS2 -> V_IN
- C66 pad 2: Net-(C66-Pad2) -> GND
- C67 pad 1: VCC -> /driver/HS2
- C67 pad 2: GND -> Net-(C67-Pad2)
- C68 pad 1: VCC -> /driver/HS2
- C68 pad 2: GND -> Net-(C68-Pad2)
- C70 pad 1: Net-(C70-Pad1) -> VCC
- C70 pad 2: /driver/HS3 -> GND
- C71 pad 1: Net-(C71-Pad1) -> VCC
- C71 pad 2: Net-(C71-Pad2) -> GND
- C72 pad 2: /driver/C_C -> /mcu/CURRENT_3
- C73 pad 1: V_IN -> Net-(C73-Pad1)
- C73 pad 2: GND -> /driver/HS3
- C74 pad 1: V_IN -> Net-(C74-Pad1)
- C74 pad 2: GND -> Net-(C74-Pad2)
- C75 pad 1: V_IN -> Net-(C75-Pad1)
- C75 pad 2: GND -> Net-(C75-Pad2)
- C77 pad 1: GND -> V_IN
- C77 pad 2: V_IN -> GND
- C79 pad 1: GND -> V_IN
- C79 pad 2: V_IN -> GND
- C82 pad 1: /driver/HS3 -> V_IN
- C82 pad 2: Net-(C82-Pad2) -> GND
- C83 pad 1: /driver/HS3 -> V_IN
- C83 pad 2: Net-(C83-Pad2) -> GND
- C9 pad 1: Net-(C9-Pad1) -> /driver/SENS_1
- C9 pad 2: GND -> Net-(C9-Pad2)
- D12 pad 1: Net-(C70-Pad1) -> Net-(C73-Pad1)
- D13 pad 1: Net-(C71-Pad1) -> Net-(C74-Pad1)
- D3 pad 1: Net-(C18-Pad1) -> Net-(C16-Pad1)
- D6 pad 1: Net-(C27-Pad1) -> Net-(C24-Pad1)
- H6 pad 1: V_IN -> (no net)
- H7 pad 1: GND -> (no net)
- NT5 pad 1: Net-(C72-Pad2) -> Net-(C75-Pad2)
- NT5 pad 2: Net-(C71-Pad2) -> Net-(C74-Pad2)
- NT6 pad 1: Net-(C72-Pad1) -> Net-(C75-Pad1)
- Q10 pad 2: Net-(C71-Pad1) -> Net-(C74-Pad1)
- Q10 pad 3: Net-(C71-Pad2) -> Net-(C74-Pad2)
- Q11 pad 1: Net-(C70-Pad1) -> Net-(C73-Pad1)
- Q12 pad 1: Net-(C71-Pad1) -> Net-(C74-Pad1)
- Q12 pad 3: Net-(C71-Pad2) -> Net-(C74-Pad2)
- Q9 pad 2: Net-(C70-Pad1) -> Net-(C73-Pad1)
- R10 pad 1: /driver/CURR_A -> /driver/SENS_2
- R10 pad 2: /driver/C_A -> /driver/HS2
- R11 pad 1: /driver/CURR_B -> /driver/SENS_2
- R11 pad 2: /driver/C_B -> GND
- R12 pad 1: /driver/SENS_2 -> /driver/SENS_3
- R12 pad 2: /driver/HS2 -> /driver/HS3
- R13 pad 1: /driver/SENS_2 -> /driver/SENS_3
- R23 pad 2: /driver/C_A -> /mcu/CURRENT_1
- R42 pad 1: Net-(R42-Pad1) -> Net-(Q6-Pad1)
- R42 pad 2: /driver/C_B -> Net-(D11-Pad2)
- R43 pad 1: /mcu/ADC_TEMP -> /driver/HO2
- R43 pad 2: VCC -> Net-(D10-Pad2)
- R44 pad 1: Net-(Q5-Pad1) -> /driver/LO2
- R44 pad 2: Net-(D10-Pad2) -> Net-(D11-Pad2)
- R45 pad 1: Net-(Q6-Pad1) -> Net-(R45-Pad1)
- R45 pad 2: Net-(D11-Pad2) -> Net-(R39-Pad1)
- R46 pad 1: /driver/HO2 -> GND
- R46 pad 2: Net-(D10-Pad2) -> /mcu/ADC_TEMP
- R47 pad 1: /driver/LO2 -> Net-(R47-Pad1)
- R47 pad 2: Net-(D11-Pad2) -> VCC
- R48 pad 1: Net-(R48-Pad1) -> Net-(C55-Pad2)
- R48 pad 2: Net-(R42-Pad1) -> Net-(R47-Pad1)
- R49 pad 1: GND -> Net-(C55-Pad1)
- R49 pad 2: /mcu/ADC_TEMP -> Net-(R45-Pad1)
- R50 pad 1: Net-(R50-Pad1) -> /driver/HS2
- R50 pad 2: VCC -> Net-(C53-Pad1)
- R51 pad 1: Net-(C55-Pad2) -> Net-(C54-Pad2)
- R51 pad 2: Net-(R50-Pad1) -> Net-(C54-Pad1)
- R52 pad 1: Net-(C55-Pad1) -> Net-(C54-Pad2)
- R52 pad 2: Net-(R48-Pad1) -> GND
- R53 pad 1: /driver/HS2 -> Net-(C67-Pad2)
- R53 pad 2: Net-(C53-Pad1) -> V_IN
- R54 pad 1: Net-(C54-Pad2) -> Net-(C68-Pad2)
- R54 pad 2: Net-(C54-Pad1) -> GND
- R55 pad 1: Net-(C54-Pad2) -> Net-(C67-Pad2)
- R55 pad 2: GND -> V_IN
- R56 pad 1: Net-(C65-Pad2) -> Net-(C68-Pad2)
- R56 pad 2: V_IN -> GND
- R57 pad 1: Net-(C66-Pad2) -> Net-(R57-Pad1)
- R57 pad 2: GND -> /mcu/CURRENT_3
- R58 pad 1: Net-(C65-Pad2) -> Net-(Q9-Pad1)
- R58 pad 2: V_IN -> Net-(D12-Pad2)
- R59 pad 1: Net-(C66-Pad2) -> Net-(Q10-Pad1)
- R59 pad 2: GND -> Net-(D13-Pad2)
- R60 pad 1: Net-(R60-Pad1) -> /driver/HO3
- R60 pad 2: /driver/C_C -> Net-(D12-Pad2)
- R61 pad 1: Net-(Q9-Pad1) -> /driver/LO3
- R61 pad 2: Net-(D12-Pad2) -> Net-(D13-Pad2)
- R62 pad 1: Net-(Q10-Pad1) -> Net-(R62-Pad1)
- R62 pad 2: Net-(D13-Pad2) -> Net-(R57-Pad1)
- R63 pad 1: /driver/HO3 -> Net-(R63-Pad1)
- R63 pad 2: Net-(D12-Pad2) -> VCC
- R64 pad 1: /driver/LO3 -> Net-(C75-Pad2)
- R64 pad 2: Net-(D13-Pad2) -> Net-(R63-Pad1)
- R65 pad 1: Net-(R65-Pad1) -> Net-(C75-Pad1)
- R65 pad 2: Net-(R60-Pad1) -> Net-(R62-Pad1)
- R66 pad 1: Net-(R66-Pad1) -> /driver/HS3
- R66 pad 2: VCC -> Net-(C73-Pad1)
- R67 pad 1: Net-(C72-Pad2) -> Net-(C74-Pad2)
- R67 pad 2: Net-(R66-Pad1) -> Net-(C74-Pad1)
- R68 pad 1: Net-(C72-Pad1) -> Net-(C74-Pad2)
- R68 pad 2: Net-(R65-Pad1) -> GND
- R69 pad 1: /driver/HS3 -> Net-(C87-Pad2)
- R69 pad 2: Net-(C70-Pad1) -> V_IN
- R70 pad 1: Net-(C71-Pad2) -> Net-(C88-Pad2)
- R70 pad 2: Net-(C71-Pad1) -> GND
- R71 pad 1: Net-(C71-Pad2) -> Net-(C87-Pad2)
- R71 pad 2: GND -> V_IN
- R72 pad 1: Net-(C82-Pad2) -> Net-(C88-Pad2)
- R72 pad 2: V_IN -> GND
- U12 pad 1: Net-(R42-Pad1) -> Net-(R39-Pad1)
- U12 pad 3: Net-(R50-Pad1) -> Net-(R47-Pad1)
- U12 pad 4: Net-(R48-Pad1) -> Net-(R45-Pad1)
- U13 pad 1: Net-(R60-Pad1) -> Net-(R57-Pad1)
- U13 pad 3: Net-(R66-Pad1) -> Net-(R63-Pad1)
- U13 pad 4: Net-(R65-Pad1) -> Net-(R62-Pad1)
- U15 pad 11: /driver/CURR_B -> /mcu/CURRENT_2
- U15 pad 16: /driver/CURR_A -> /mcu/CURRENT_1
- U15 pad 2: /driver/CURR_FILTER -> unconnected-(U15-Pad2)
- U15 pad 40: unconnected-(U15-Pad40) -> /driver/SENS_FILTER
- U15 pad 8: /driver/CURR_C -> /mcu/CURRENT_3
- U3 pad 1: /driver/CURR_A -> Net-(C9-Pad2)
- U3 pad 2: Net-(C9-Pad1) -> GND
- U3 pad 4: /driver/CURR_FILTER -> /driver/SENS_FILTER
- U5 pad 1: /driver/CURR_B -> Net-(C14-Pad2)
- U5 pad 2: Net-(C15-Pad1) -> GND
- U5 pad 4: /driver/CURR_FILTER -> /driver/SENS_FILTER
- U7 pad 8: Net-(C18-Pad1) -> Net-(C16-Pad1)
- U8 pad 1: /driver/CURR_C -> Net-(C17-Pad2)
- U8 pad 2: Net-(C20-Pad1) -> GND
- U8 pad 4: /driver/CURR_FILTER -> /driver/SENS_FILTER
- U9 pad 8: Net-(C27-Pad1) -> Net-(C24-Pad1)
Routing:
- net GND: track 71.8 -> 20.8 mm, vias 912 -> 1162
- net /driver/SENS_FILTER: track 0.00 -> 47.6 mm, vias 0 -> 6
- net /mcu/CURRENT_3: track 0.00 -> 38.5 mm
- net /driver/C_C: track 37.8 -> 0.00 mm
- net /driver/HS1: track 6.78 -> 40.4 mm
- net Net-(C75-Pad1): track 0.00 -> 26.6 mm, vias 0 -> 1
- net /mcu/CURRENT_2: track 0.00 -> 26.4 mm
- net Net-(C75-Pad2): track 0.00 -> 26.2 mm, vias 0 -> 1
- net /driver/HS2: track 14.3 -> 40.3 mm
- net /driver/HS3: track 14.4 -> 40.4 mm
- net Net-(C72-Pad1): track 25.9 -> 0.00 mm, vias 1 -> 0
- net Net-(C72-Pad2): track 25.6 -> 0.00 mm
- net /driver/C_B: track 24.9 -> 0.00 mm
- net /driver/H1: track 80.2 -> 56.6 mm, vias 0 -> 6
- net /mcu/CURRENT_1: track 0.00 -> 18.3 mm
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- removed copper zone on F.Cu, net /driver/HS1
- removed copper zone on F.Cu, net /driver/HS2
- removed copper zone on F.Cu, net /driver/HS3
- removed copper zone on B.Cu, net /mcu/ADC_TEMP
- removed copper zone on F.Cu, net /mcu/ADC_TEMP
- removed copper zone on F.Cu, net V_IN
Other:
- board size 60.7 x 89.9 mm -> 62.2 x 90.8 mm
- board text added: "++++"
- board text added: "----"
- board text removed: "++++++"
- board text removed: "------"
- board text removed: "{"

Commit message: Add files via upload
Parts:
- removed the C91 at (82.9, 121.9)
- removed the C92 at (91.0, 120.1)
- removed the C93 at (98.6, 123.6)
- moved R39 0.23 mm to (99.1, 112.4)
- moved C9 0.12 mm to (81.6, 121.9)
- renumbered C106 to C100, C107 to C101, C108 to C102, C109 to C103, C110 to C104, C49 to C48, C50 to C49, C51 to C50, C52 to C51, C53 to C52, C54 to C53, C55 to C54, C56 to C55, C57 to C56, C58 to C57, C59 to C58, C60 to C59, C61 to C60, C62 to C61, C63 to C62, C64 to C63, C65 to C64, C66 to C65, C67 to C66, C68 to C67, C70 to C68, C71 to C69, C72 to C70, C73 to C71, C74 to C72, C75 to C73, C76 to C74, C77 to C75, C78 to C76, C79 to C77, C80 to C78, C81 to C79, C82 to C80, C83 to C81, C84 to C82, C85 to C83, C86 to C84, C87 to C85, C88 to C86, C90 to C87, C94 to C88, C95 to C89, C96 to C90, C97 to C91, C98 to C92, C99 to C93, C100 to C94, C101 to C95, C102 to C96, C103 to C97, C104 to C98, C105 to C99
Routing:
- net +5V: track 127.0 -> 125.7 mm
- net /mcu/CAN_RX: track 27.9 -> 26.8 mm
- net +12V: track 266.5 -> 265.5 mm
- net /mcu/CAN_TX: track 23.4 -> 22.9 mm
- net GND: vias 1162 -> 1161
