File: source/foc.kicad_sch (KiCad schematic)
At the start: 7 parts, among them P1 SWD, U1 BMI160

Commit message: Add files via upload
Parts:
- removed FieldFeets1: R, Custom:field, symbol Device:R
- added H1, H2, H3, H4, H5, H6: MountingHole, MountingHole:MountingHole_3.2mm_M3, symbol Mechanical:MountingHole
Other:
- note added: "Mounting Holes"

Commit message: Add files via upload
Parts:
- added H7: MountingHole, MountingHole:MountingHole_3.2mm_M3, symbol Mechanical:MountingHole
- added H8: MountingHole, MountingHole:MountingHole_3.7mm, symbol Mechanical:MountingHole
- H2, H4, H6: footprint MountingHole:MountingHole_3.2mm_M3 -> MountingHole:MountingHole_3.7mm
Other:
- note added: "WATT'EVER"
- note removed: "F-Of-C"

Commit message: Add files via upload
Parts:
- removed H2, H4, H6, H8: MountingHole, MountingHole:MountingHole_3.7mm, symbol Mechanical:MountingHole
- added H3: MountingHole, MountingHole:MountingHole_3.2mm_M3, symbol Mechanical:MountingHole
- renumbered H3 to H2, H7 to H4
Other:
- note removed: "Connect signal ground and power ground in one place only"

Commit message: Add files via upload
Parts:
- added C3: 100n, Resistor_SMD:R_0603_1608Metric, symbol Device:C
- added J1: Conn_01x06, Connector_JST:JST_PH_B6B-PH-K_1x06_P2.00mm_Vertical, symbol Connector_Generic:Conn_01x06
- added J2: Conn_01x08, Connector_JST:JST_PH_B8B-PH-K_1x08_P2.00mm_Vertical, symbol Connector_Generic:Conn_01x08
- added J3: NRF wireless, Connector_PinSocket_2.54mm:PinSocket_2x04_P2.54mm_Vertical, symbol Connector_Generic:Conn_02x04_Odd_Even
- added R1, R2, R3: 2k2, Resistor_SMD:R_0603_1608Metric, symbol Device:R
- added R5: 10k, Resistor_SMD:R_0603_1608Metric, symbol Device:R
- added SW1: SW_DPDT_x2, Jumper:SolderJumper-3_P1.3mm_Bridged2Bar12_Pad1.0x1.5mm, symbol Switch:SW_DPDT_x2
- renumbered R1 to R4, R2 to R6
Connections:
- net GND: now also C3.2, J1.1 (Pin_1), J2.3 (Pin_3), J3.2 (Pin_2)
- net VCC: now also J2.2 (Pin_2), J3.1 (Pin_1), J3.4 (Pin_4), R5.2, SW1.1 (A)
- net mcu/HALL_1: now also J1.4 (Pin_4), R1.2
- net mcu/HALL_2: now also J1.3 (Pin_3), R2.2
- net mcu/HALL_3: now also J1.2 (Pin_2), R3.2
- net mcu/TEMP_MOTOR: now also C3.1, J1.5 (Pin_5), R5.1
- new net: J1.6 (Pin_6), R1.1, R2.1, R3.1, SW1.2 (B)
- new net +5V: J2.1 (Pin_1), SW1.3 (C)
- new net mcu/ADC_15: J2.8 (Pin_8)
- new net mcu/MISO_ADC_EXT2: J2.7 (Pin_7)
- new net mcu/NRF_CSN: J3.3 (Pin_3)
- new net mcu/NRF_MISO: J3.8 (Pin_8)
- new net mcu/NRF_MOSI: J3.5 (Pin_5)
- new net mcu/NRF_SCK: J3.6 (Pin_6)
- new net mcu/RX_SDA_NSS: J2.5 (Pin_5)
- new net mcu/SCK_ADC_EXT: J2.4 (Pin_4)
- new net mcu/TX_SCL_MOSI: J2.6 (Pin_6)
- no-connect marks 22 -> 19
Other:
- sheet mcu ports: added ADC_15, MISO_ADC_EXT2, NRF_CSN, NRF_MISO, NRF_MOSI, NRF_SCK, RX_SDA_NSS, SCK_ADC_EXT, TX_SCL_MOSI; removed none
- moved on the sheet: H2, H3, H4, H5, P1

Commit message: Add files via upload
Parts:
- added C3: 100n, Resistor_SMD:R_0603_1608Metric, symbol Device:C
- added J1: Conn_01x03, Connector_JST:JST_PH_B3B-PH-K_1x03_P2.00mm_Vertical, symbol Connector_Generic:Conn_01x03
- added R4: 100R, Resistor_SMD:R_0603_1608Metric, symbol Device:R_Small
- renumbered C3 to C4, J1 to J2, J2 to J3, J3 to J4, R4 to R5, R5 to R6, R6 to R7
Connections:
- net +5V: now also J1.2 (Pin_2)
- net GND: now also C3.2, J1.3 (Pin_3)
- net VCC: now also P1.1 (Pin_1); no longer P1.5 (Pin_5)
- net mcu/NRST: now also P1.5 (Pin_5); no longer P1.1 (Pin_1)
- net mcu/SERVO: now also C3.1, R4.1
- net mcu/SWCLK: now also P1.2 (Pin_2); no longer P1.4 (Pin_4)
- net mcu/SWDIO: now also P1.4 (Pin_4); no longer P1.2 (Pin_2)
- new net: J1.1 (Pin_1), R4.2
- no-connect marks 19 -> 17
Other:
- sheet driver ports: added CURR_A, CURR_B, CURR_C, CURR_FILTER, C_A, C_B, C_C; removed none
- sheet mcu ports: added CURR_FILTER; removed VDO_I
- sheet power ports: added C_A, C_B, C_C; removed CURR_A, CURR_B, CURR_C
- moved on the sheet: P1

Commit message: Add files via upload
Parts:
- added H6, H7, H8: MountingHole, MountingHole:MountingHole_4.3mm_M4_Pad_TopOnly, symbol Mechanical:MountingHole
Other:
- sheet driver ports: added SENS_FILTER; removed CURR_A, CURR_B, CURR_C, CURR_FILTER, C_A, C_B, C_C
- sheet mcu ports: added VOLTAGE_FILTER; removed CURR_FILTER
- sheet power ports: added CURR_A, CURR_B, CURR_C; removed C_A, C_B, C_C
- note added: "FOC KING"
- note removed: "WATT'EVER"
