File: source/mcu.kicad_sch (KiCad schematic)
At the start: 45 parts, among them J1 Conn_01x04_Male, J2 TYPE-C-31-M-12, U10 HT7550, U11 STM32F405RGT6, U12 AMS1117-3.3, U9 TJA1050T/CM,118, Y1 8MHz Crystal Resonator, X5032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

Commit message: Add files via upload
Parts:
- renumbered C98 to C100, C99 to C101, C100 to C102, C101 to C103, C102 to C104, C103 to C105, C104 to C106, C105 to C107, C106 to C108, C107 to C109, C108 to C110, C82 to C84, C83 to C85, C84 to C86, C85 to C87, C86 to C88, C87 to C89, C88 to C90, C89 to C91, C90 to C92, C91 to C93, C93 to C94, C92 to C95, C94 to C96, C95 to C97, C96 to C98, C97 to C99, R53 to R59, R54 to R60, R55 to R61, R56 to R62, R57 to R63, R58 to R64, R59 to R65

Commit message: Add files via upload
Parts:
- removed C102, C97: 100n, Capacitor_SMD:C_0603_1608Metric, symbol Device:C_Small
- removed C110: 2.2u, Capacitor_SMD:C_0603_1608Metric, symbol BLDC_4-rescue:C-RESCUE-BLDC_4
Other:
- moved on the sheet: C103, C99

Commit message: Add files via upload
Parts:
- renumbered C84 to C67, C85 to C68, C86 to C69, C87 to C70, C88 to C71, C89 to C72, C90 to C73, C91 to C74, C92 to C75, C93 to C76, C94 to C77, C95 to C78, C96 to C79, C99 to C80, C98 to C81, C103 to C82, C100 to C83, C101 to C84, C104 to C85, C105 to C86, C106 to C87, C107 to C88, C108 to C89, C109 to C90, D16 to D10, D17 to D11, D18 to D12, R59 to R65, R60 to R66, R61 to R67, R62 to R68, R63 to R69, R64 to R70, R65 to R71
Other:
- note added: "WATT'EVER"
- note removed: "F-Of-C"

Commit message: Add files via upload
Parts:
- renumbered C67 to C73, C68 to C74, C69 to C75, C70 to C76, C71 to C77, C72 to C78, C73 to C79, C74 to C80, C75 to C81, C76 to C82, C77 to C83, C78 to C84, C79 to C85, C80 to C86, C81 to C87, C82 to C88, C83 to C89, C84 to C90, C85 to C91, C86 to C92, C87 to C93, C88 to C94, C89 to C95, C90 to C96

Commit message: Add files via upload
Parts:
- renumbered J1 to J4, J2 to J5, R65 to R69, R66 to R70, R67 to R71, R68 to R72, R69 to R73, R70 to R74, R71 to R75
Connections:
- net LED_RED: now also U11.58 (PB6); no longer U11.59 (PB7)
- net SERVO: now also U11.51 (PC10); no longer U11.58 (PB6)
- net RX_SDA_NSS: now reaches U11.20 (PA4(ADC12_IN4/DAC1_OUT))
- net SCK_ADC_EXT: now reaches U11.21 (PA5(ADC12_IN5/DAC2_OUT))
- net MISO_ADC_EXT2: now reaches U11.22 (PA6(ADC12_IN6))
- net TX_SCL_MOSI: now reaches U11.23 (PA7(ADC12_IN7))
- net ADC_15: now reaches U11.25 (PC5(ADC12_IN15))
- net NRF_MISO: now reaches U11.54 (PD2)
- net NRF_MOSI: now reaches U11.55 (PB3(JTDO/TRACESWO))
- net NRF_SCK: now reaches U11.56 (PB4(NJTRST))
- new net NRF_CSN: U11.59 (PB7)
- no-connect marks 23 -> 14

Commit message: Add files via upload
Parts:
- removed C79, C96: 10u, Capacitor_Tantalum_SMD:CP_EIA-3216-10_Kemet-I, symbol Device:C_Polarized_Small
- removed C92: 100n, Capacitor_SMD:C_0603_1608Metric, symbol BLDC_4-rescue:C-RESCUE-BLDC_4
- removed U10: HT7550, Package_TO_SOT_SMD:SOT-89-3, symbol Regulator_Linear:L79L08_SOT89
- removed U12: AMS1117-3.3, Package_TO_SOT_SMD:SOT-223-3_TabPin2, symbol Regulator_Linear:LM1117-3.3
- R76: renamed from R69; value 100Ω -> 100R
- R77: renamed from R70; value 100Ω -> 100R
- R80: renamed from R73; value 20k -> 10k; LCSC C4184 -> C25804
- R81: renamed from R74; value 20k -> 10k; LCSC C4184 -> C25804
- renumbered C90 to C100, C91 to C101, C93 to C102, C94 to C103, C95 to C104, C73 to C84, C74 to C85, C75 to C86, C76 to C87, C77 to C88, C78 to C89, C80 to C90, C81 to C91, C82 to C92, C83 to C93, C84 to C94, C85 to C95, C86 to C96, C87 to C97, C88 to C98, C89 to C99, D10 to D14, D11 to D15, D12 to D16, J4 to J5, J5 to J6, R71 to R78, R72 to R79, R75 to R82, U9 to U14, U11 to U15
Connections:
- net +5V: no longer J6.A4B9 (VBUS), J6.B4A9 (VBUS)
- net RX_SDA_NSS: now also U15.30 (PB11)
- net SERVO: now also U15.27 (PB1(ADC12_IN9)); no longer U15.51 (PC10)
- net TX_SCL_MOSI: now also U15.29 (PB10)
- net CURR_FILTER: now reaches U15.2 (PC13_(RTC_AF1))
- no-connect marks 14 -> 13
Other:
- note added: "TIM3_CH4 is configured for pin PB1 pin 27 according to stm32f405 datasheet https://www.st.com/en/microcontrollers-microprocessors/stm32f405rg.html"
- note removed: "BOARD REGULATOR"
- note removed: "CAN REGULATOR"
- moved on the sheet: C84

Commit message: Add files via upload
Parts:
- renumbered C94 to C100, C95 to C101, C96 to C102, C97 to C103, C98 to C104, C99 to C105, C100 to C106, C101 to C107, C102 to C108, C103 to C109, C104 to C110, C84 to C90, C85 to C91, C86 to C92, C87 to C93, C88 to C94, C89 to C95, C90 to C96, C91 to C97, C92 to C98, C93 to C99, R76 to R73, R77 to R74, R78 to R75, R79 to R76, R80 to R77, R81 to R78, R82 to R79
Connections:
- net VOLTAGE_FILTER: now reaches U15.40 (PC9)
- net CURR_FILTER: no longer names the net of U15.2 (PC13_(RTC_AF1))
Other:
- note added: "FOC KING"
- note removed: "WATT'EVER"
Changed lines of the file:
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@@
   (no_connect (at 157.48 43.18))
   (no_connect (at 93.98 139.7))
+  (no_connect (at 93.98 144.78))
   (no_connect (at 93.98 142.24))
   (no_connect (at 200.66 146.05))
   (no_connect (at 93.98 99.06))
-  (no_connect (at 93.98 134.62))
   (no_connect (at 77.47 180.34))
   (no_connect (at 236.22 139.7))
@@
     (effects (font (size 1.27 1.27)) (justify left bottom))
   )
-  (text "WATT'EVER" (at 187.96 191.77 0)
+  (text "FOC KING" (at 187.96 191.77 0)
     (effects (font (size 2.54 2.54)) (justify left bottom))
   )
@@
     (effects (font (size 1.524 1.524)) (justify left))
   )
+  (hierarchical_label "VOLTAGE_FILTER" (shape output) (at 93.98 134.62 180)
+    (effects (font (size 1.27 1.27)) (justify right))
+  )
   (hierarchical_label "USB_D+" (shape bidirectional) (at 200.66 140.97 180)
     (effects (font (size 1.524 1.524)) (justify right))
@@
     (effects (font (size 1.524 1.524)) (justify right))
   )
-  (hierarchical_label "CURR_FILTER" (shape output) (at 93.98 144.78 180)
-    (effects (font (size 1.27 1.27)) (justify right))
-  )
   (hierarchical_label "NRF_MOSI" (shape input) (at 157.48 80.01 0)
     (effects (font (size 1.27 1.27)) (justify left))
@@
   (symbol (lib_id "Device:C_Small") (at 218.44 25.4 0) (unit 1)
     (in_bom yes) (on_board yes)
-    (property "Reference" "C98" (id 0) (at 220.98 24.13 0)
+    (property "Reference" "C104" (id 0) (at 220.98 24.13 0)
       (effects (font (size 1.27 1.27)) (justify left))
     )
@@
   (symbol (lib_id "Device:R_Small") (at 40.64 176.53 0) (mirror x) (unit 1)
     (in_bom yes) (on_board yes)
-    (property "Reference" "R76" (id 0) (at 39.37 175.26 0)
+    (property "Reference" "R73" (id 0) (at 39.37 175.26 0)
       (effects (font (size 1.27 1.27)) (justify right))
     )
@@
   (symbol (lib_id "Device:R_Small") (at 245.11 107.95 180) (unit 1)
     (in_bom yes) (on_board yes)
-    (property "Reference" "R80" (id 0) (at 237.49 107.95 0)
+    (property "Reference" "R77" (id 0) (at 237.49 107.95 0)
       (effects (font (size 1.27 1.27)) (justify right))
     )
@@
   (symbol (lib_id "Device:C_Small") (at 48.26 176.53 0) (mirror y) (unit 1)
     (in_bom yes) (on_board yes)
-    (property "Reference" "C88" (id 0) (at 45.72 175.26 0)
+    (property "Reference" "C94" (id 0) (at 45.72 175.26 0)
       (effects (font (size 1.27 1.27)) (justify left))
     )
@@
   (symbol (lib_id "BLDC_4-rescue:C-RESCUE-BLDC_4") (at 273.05 30.48 180) (unit 1)
     (in_bom yes) (on_board yes)
-    (property "Reference" "C104" (id 0) (at 271.78 33.02 0)
+    (property "Reference" "C110" (id 0) (at 271.78 33.02 0)
       (effects (font (size 1.27 1.27)) (justify left))
     )
@@
   (symbol (lib_id "Device:C_Small") (at 198.12 25.4 0) (unit 1)
     (in_bom yes) (on_board yes)
-    (property "Reference" "C95" (id 0) (at 200.66 24.13 0)
+    (property "Reference" "C101" (id 0) (at 200.66 24.13 0)
       (effects (font (size 1.27 1.27)) (justify left))
     )
@@
   (symbol (lib_id "Device:R_Small") (at 196.85 138.43 270) (unit 1)
     (in_bom yes) (on_board yes)
-    (property "Reference" "R78" (id 0) (at 193.04 135.89 90))
+    (property "Reference" "R75" (id 0) (at 193.04 135.89 90))
     (property "Value" "5.1k" (id 1) (at 199.39 135.89 90))
     (property "Footprint" "Resistor_SMD:R_0603_1608Metric" (id 2) (at 196.85 138.43 0)
@@
   (symbol (lib_id "BLDC_4-rescue:C-RESCUE-BLDC_4") (at 266.7 30.48 180) (unit 1)
     (in_bom yes) (on_board yes)
-    (property "Reference" "C103" (id 0) (at 265.43 33.02 0)
+    (property "Reference" "C109" (id 0) (at 265.43 33.02 0)
       (effects (font (size 1.27 1.27)) (justify left))
     )
@@
   (symbol (lib_id "Device:C_Small") (at 189.23 25.4 0) (unit 1)
     (in_bom yes) (on_board yes)
-    (property "Reference" "C94" (id 0) (at 191.77 24.13 0)
+    (property "Reference" "C100" (id 0) (at 191.77 24.13 0)
       (effects (font (size 1.27 1.27)) (justify left))
     )
@@
   (symbol (lib_id "Device:C_Small") (at 208.28 25.4 0) (unit 1)
     (in_bom yes) (on_board yes)
-    (property "Reference" "C96" (id 0) (at 210.82 24.13 0)
+    (property "Reference" "C102" (id 0) (at 210.82 24.13 0)
       (effects (font (size 1.27 1.27)) (justify left))
     )
@@
   (symbol (lib_id "Device:R_Small") (at 251.46 107.95 180) (unit 1)
     (in_bom yes) (on_board yes)
-    (property "Reference" "R81" (id 0) (at 252.984 107.442 0)
+    (property "Reference" "R78" (id 0) (at 252.984 107.442 0)
       (effects (font (size 1.27 1.27)) (justify right))
     )
@@
   (symbol (lib_id "Device:R_Small") (at 40.64 184.15 0) (mirror x) (unit 1)
     (in_bom yes) (on_board yes)
-    (property "Reference" "R77" (id 0) (at 40.64 181.61 0)
+    (property "Reference" "R74" (id 0) (at 40.64 181.61 0)
       (effects (font (size 1.27 1.27)) (justify right))
     )
@@
   (symbol (lib_id "Device:C_Small") (at 38.1 38.1 0) (unit 1)
     (in_bom yes) (on_board yes)
-    (property "Reference" "C85" (id 0) (at 40.64 36.83 0)
+    (property "Reference" "C91" (id 0) (at 40.64 36.83 0)
       (effects (font (size 1.27 1.27)) (justify left))
     )
@@
   (symbol (lib_id "Device:C_Small") (at 158.75 156.21 0) (unit 1)
     (in_bom yes) (on_board yes)
-    (property "Reference" "C90" (id 0) (at 149.86 156.21 0)
+    (property "Reference" "C96" (id 0) (at 149.86 156.21 0)
       (effects (font (size 1.27 1.27)) (justify left))
     )
@@
   (symbol (lib_id "Device:C_Small") (at 165.1 153.67 0) (unit 1)
     (in_bom yes) (on_board yes)
-    (property "Reference" "C91" (id 0) (at 168.275 151.765 0)
+    (property "Reference" "C97" (id 0) (at 168.275 151.765 0)
       (effects (font (size 1.27 1.27)) (justify left))
     )
@@
   (symbol (lib_id "Device:C_Small") (at 38.1 60.96 0) (unit 1)
     (in_bom yes) (on_board yes)
-    (property "Reference" "C87" (id 0) (at 40.64 59.69 0)
+    (property "Reference" "C93" (id 0) (at 40.64 59.69 0)
       (effects (font (size 1.27 1.27)) (justify left))
     )
@@
   (symbol (lib_id "Device:C_Small") (at 50.8 190.5 0) (mirror y) (unit 1)
     (in_bom yes) (on_board yes)
-    (property "Reference" "C89" (id 0) (at 48.26 189.23 0)
+    (property "Reference" "C95" (id 0) (at 48.26 189.23 0)
       (effects (font (size 1.27 1.27)) (justify left))
     )
@@
   (symbol (lib_id "BLDC_4-rescue:C-RESCUE-BLDC_4") (at 260.35 30.48 180) (unit 1)
     (in_bom yes) (on_board yes)
-    (property "Reference" "C102" (id 0) (at 259.08 33.02 0)
+    (property "Reference" "C108" (id 0) (at 259.08 33.02 0)
       (effects (font (size 1.27 1.27)) (justify left))
     )
@@
   (symbol (lib_id "Device:C_Small") (at 213.36 42.545 0) (unit 1)
     (in_bom yes) (on_board yes)
-    (property "Reference" "C97" (id 0) (at 215.9 41.275 0)
+    (property "Reference" "C103" (id 0) (at 215.9 41.275 0)
       (effects (font (size 1.27 1.27)) (justify left))
     )
@@
   (symbol (lib_id "Device:C_Small") (at 180.34 25.4 0) (unit 1)
     (in_bom yes) (on_board yes)
-    (property "Reference" "C92" (id 0) (at 182.88 24.13 0)
+    (property "Reference" "C98" (id 0) (at 182.88 24.13 0)
       (effects (font (size 1.27 1.27)) (justify left))
     )
@@
   (symbol (lib_id "Device:C_Small") (at 34.29 182.88 0) (mirror y) (unit 1)
     (in_bom yes) (on_board yes)
-    (property "Reference" "C84" (id 0) (at 33.02 180.34 0)
+    (property "Reference" "C90" (id 0) (at 33.02 180.34 0)
       (effects (font (size 1.27 1.27)) (justify left))
     )
@@
   (symbol (lib_id "Device:R_Small") (at 240.03 147.32 90) (unit 1)
     (in_bom yes) (on_board yes)
-    (property "Reference" "R79" (id 0) (at 241.3 149.86 90))
+    (property "Reference" "R76" (id 0) (at 241.3 149.86 90))
     (property "Value" "5.1k" (id 1) (at 236.22 148.59 90))
     (property "Footprint" "Resistor_SMD:R_0603_1608Metric" (id 2) (at 240.03 147.32 0)
@@
   (symbol (lib_id "BLDC_4-rescue:C-RESCUE-BLDC_4") (at 181.61 74.93 180) (unit 1)
     (in_bom yes) (on_board yes)
-    (property "Reference" "C93" (id 0) (at 185.42 72.39 0)
+    (property "Reference" "C99" (id 0) (at 185.42 72.39 0)
       (effects (font (size 1.27 1.27)) (justify left))
     )
@@
   (symbol (lib_id "Device:C_Small") (at 241.3 68.58 0) (unit 1)
     (in_bom yes) (on_board yes)
-    (property "Reference" "C101" (id 0) (at 234.95 71.12 0)
+    (property "Reference" "C107" (id 0) (at 234.95 71.12 0)
       (effects (font (size 1.27 1.27)) (justify left))
     )
@@
   (symbol (lib_id "Device:R_Small") (at 257.81 108.077 180) (unit 1)
     (in_bom yes) (on_board yes)
-    (property "Reference" "R82" (id 0) (at 258.953 107.442 0)
+    (property "Reference" "R79" (id 0) (at 258.953 107.442 0)
       (effects (font (size 1.27 1.27)) (justify right))
     )
@@
   (symbol (lib_id "Device:C_Small") (at 38.1 49.53 0) (unit 1)
     (in_bom yes) (on_board yes)
-    (property "Reference" "C86" (id 0) (at 40.64 48.26 0)
+    (property "Reference" "C92" (id 0) (at 40.64 48.26 0)
       (effects (font (size 1.27 1.27)) (justify left))
     )
@@
   (symbol (lib_id "Device:C_Small") (at 222.25 42.545 0) (unit 1)
     (in_bom yes) (on_board yes)
-    (property "Reference" "C99" (id 0) (at 224.79 41.275 0)
+    (property "Reference" "C105" (id 0) (at 224.79 41.275 0)
       (effects (font (size 1.27 1.27)) (justify left))
     )
@@
   (symbol (lib_id "Device:C_Small") (at 226.06 68.58 0) (unit 1)
     (in_bom yes) (on_board yes)
-    (property "Reference" "C100" (id 0) (at 220.98 71.12 0)
+    (property "Reference" "C106" (id 0) (at 220.98 71.12 0)
       (effects (font (size 1.27 1.27)) (justify left))
     )

Commit message: Add files via upload
Parts:
- removed C91, C92, C93: 100n, Capacitor_SMD:C_0603_1608Metric, symbol Device:C_Small
- renumbered C106 to C100, C107 to C101, C108 to C102, C109 to C103, C110 to C104, C90 to C87, C94 to C88, C95 to C89, C96 to C90, C97 to C91, C98 to C92, C99 to C93, C100 to C94, C101 to C95, C102 to C96, C103 to C97, C104 to C98, C105 to C99
Other:
- note removed: "VSENSE FILTERS"
