File: source/power.kicad_sch (KiCad schematic)
At the start: 123 parts, among them Q1 MMBT5401, Q10 CSD19536KCS, Q11 CSD19536KCS, Q12 CSD19536KCS, Q13 MMBT5401, Q14 MMBT5401, Q15 CSD19536KCS, Q16 CSD19536KCS, Q17 CSD19536KCS, Q18 CSD19536KCS, Q2 MMBT5401, Q3 NCEP60T20, Q4 CSD19536KCS, Q5 CSD19536KCS, Q6 CSD19536KCS, Q7 MMBT5401, Q8 MMBT5401, Q9 CSD19536KCS, U6 MS8311, U7 MS8311, U8 MS8311

Commit message: Add files via upload
Parts:
- added C39, C41, C61, C63, C82, C83: 4.7n, Capacitor_SMD:C_0603_1608Metric, symbol Device:C
- added R31, R32, R45, R46, R57, R58: 10R, Resistor_SMD:R_0603_1608Metric, symbol Device:R
- renumbered C24 to C20, C25 to C21, C26 to C22, C27 to C23, C28 to C24, C29 to C25, C30 to C26, C31 to C27, C32 to C28, C33 to C29, C34 to C30, C35 to C31, C36 to C32, C37 to C33, C38 to C34, C39 to C35, C40 to C36, C41 to C37, C42 to C38, C43 to C40, C44 to C42, C45 to C43, C46 to C44, C47 to C45, C48 to C46, C49 to C47, C50 to C48, C51 to C49, C52 to C50, C53 to C51, C54 to C52, C55 to C53, C56 to C54, C57 to C55, C58 to C56, C59 to C57, C60 to C58, C61 to C59, C62 to C60, C64 to C62, C63 to C64, R31 to R33, R32 to R34, R33 to R35, R34 to R36, R35 to R37, R36 to R38, R37 to R39, R38 to R40, R39 to R41, R40 to R42, R41 to R43, R42 to R44, R43 to R47, R44 to R48, R45 to R49, R46 to R50, R47 to R51, R48 to R52, R49 to R53, R50 to R54, R51 to R55, R52 to R56
Connections:
- net GND: now also R31.2, R32.2, R45.2, R46.2, R57.2, R58.2
- net SH_A: now also C39.2
- net SH_B: now also C61.2
- net SH_C: now also C82.2
- new net: C41.2, R31.1, R32.1
- new net: C61.1, C63.1
- new net: C63.2, R45.1, R46.1
- new net: C82.1, C83.1
- new net: C83.2, R57.1, R58.1
- new net: C39.1, C41.1
Other:
- note added: "Snubber A"
- note added: "Snubber B"
- note added: "Snubber C"

Commit message: Add files via upload
Parts:
- R34: footprint Resistor_SMD:R_0402_1005Metric -> Resistor_SMD:R_0603_1608Metric
- R38: footprint Resistor_SMD:R_0402_1005Metric -> Resistor_SMD:R_0603_1608Metric; LCSC C25744 -> C25804
Changed lines of the file:
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@@
     (property "Reference" "R38" (id 0) (at 134.62 166.37 90))
     (property "Value" "10k" (id 1) (at 134.62 168.91 90))
-    (property "Footprint" "Resistor_SMD:R_0402_1005Metric" (id 2) (at 134.62 167.132 90)
+    (property "Footprint" "Resistor_SMD:R_0603_1608Metric" (id 2) (at 134.62 167.132 90)
       (effects (font (size 1.27 1.27)) hide)
     )
@@
       (effects (font (size 1.27 1.27)) hide)
     )
-    (property "LCSC" "C25744" (id 4) (at 134.62 168.91 90)
+    (property "LCSC" "C25804" (id 4) (at 134.62 168.91 90)
       (effects (font (size 1.27 1.27)) hide)
     )
@@
     (property "Reference" "R34" (id 0) (at 123.19 166.37 90))
     (property "Value" "NTC 10k" (id 1) (at 123.19 171.45 90))
-    (property "Footprint" "Resistor_SMD:R_0402_1005Metric" (id 2) (at 123.19 167.132 90)
-      (effects (font (size 1.27 1.27)) hide)
-    )
+    (property "Footprint" "Resistor_SMD:R_0603_1608Metric" (id 2) (at 123.19 167.132 90)
+      (effects (font (size 1.27 1.27)) hide)
+    )

Commit message: Add files via upload
Parts:
- removed C26, C28, C29, C30, C32, C33, C34, C36, C37, C48, C50, C51, C52, C54, C55, C56, C58, C59, C69, C71, C72, C73, C75, C76, C77, C79, C80: 10u @ 50V, Capacitor_SMD:C_1206_3216Metric, symbol BLDC_4-rescue:C-RESCUE-BLDC_4
- removed C39, C61, C82: 4.7n, Capacitor_SMD:C_0603_1608Metric, symbol Device:C
- removed D10, D11, D12, D13, D14, D15: 1N4148WS, Diode_SMD:D_SOD-323, symbol Diode:1N4148W
- removed Q1, Q13, Q14, Q2, Q7, Q8: MMBT5401, Package_TO_SOT_SMD:SOT-23, symbol Device:Q_PNP_BEC
- added C34, C50, C65: 4.7n, Capacitor_SMD:C_0603_1608Metric, symbol Device:C
- added R31, R33, R47, R49, R61, R63: 10R, Resistor_SMD:R_0603_1608Metric, symbol Device:R
- C27: value 10u @ 50V -> 10u @ 100V; footprint Capacitor_SMD:C_1206_3216Metric -> Capacitor_SMD:C_2220_5650Metric; LCSC C13585 -> C2843466
- C29: renamed from C31; value 10u @ 50V -> 10u @ 100V; footprint Capacitor_SMD:C_1206_3216Metric -> Capacitor_SMD:C_2220_5650Metric; LCSC C13585 -> C2843466
- C31: renamed from C35; value 10u @ 50V -> 10u @ 100V; footprint Capacitor_SMD:C_1206_3216Metric -> Capacitor_SMD:C_2220_5650Metric; LCSC C13585 -> C2843466
- C35: renamed from C41; LCSC C53987 -> C382251
- C43: renamed from C49; value 10u @ 50V -> 10u @ 100V; footprint Capacitor_SMD:C_1206_3216Metric -> Capacitor_SMD:C_2220_5650Metric; LCSC C13585 -> C2843466
- C45: renamed from C53; value 10u @ 50V -> 10u @ 100V; footprint Capacitor_SMD:C_1206_3216Metric -> Capacitor_SMD:C_2220_5650Metric; LCSC C13585 -> C2843466
- C47: renamed from C57; value 10u @ 50V -> 10u @ 100V; footprint Capacitor_SMD:C_1206_3216Metric -> Capacitor_SMD:C_2220_5650Metric; LCSC C13585 -> C2843466
- C51: renamed from C63; LCSC C53987 -> C382251
- C58: renamed from C70; value 10u @ 50V -> 10u @ 100V; footprint Capacitor_SMD:C_1206_3216Metric -> Capacitor_SMD:C_2220_5650Metric; LCSC C13585 -> C2843466
- C60: renamed from C74; value 10u @ 50V -> 10u @ 100V; footprint Capacitor_SMD:C_1206_3216Metric -> Capacitor_SMD:C_2220_5650Metric; LCSC C13585 -> C2843466
- C62: renamed from C78; value 10u @ 50V -> 10u @ 100V; footprint Capacitor_SMD:C_1206_3216Metric -> Capacitor_SMD:C_2220_5650Metric; LCSC C13585 -> C2843466
- C66: renamed from C83; LCSC C53987 -> C382251
- renumbered C20 to C21, C21 to C22, C22 to C23, C23 to C24, C24 to C25, C25 to C26, C38 to C33, C40 to C36, C42 to C37, C43 to C38, C44 to C39, C45 to C40, C46 to C41, C47 to C42, C60 to C49, C62 to C52, C64 to C53, C65 to C54, C66 to C55, C67 to C56, C68 to C57, C81 to C64, Q3 to Q1, Q16 to Q10, Q17 to Q11, Q18 to Q12, Q4 to Q2, Q5 to Q3, Q6 to Q4, Q9 to Q5, Q10 to Q6, Q11 to Q7, Q12 to Q8, Q15 to Q9, R31 to R32, R32 to R34, R33 to R35, R34 to R36, R35 to R37, R36 to R38, R37 to R39, R38 to R40, R39 to R41, R40 to R42, R41 to R43, R42 to R44, R43 to R45, R44 to R46, R45 to R48, R46 to R50, R47 to R51, R48 to R52, R49 to R53, R50 to R54, R51 to R55, R52 to R56, R53 to R57, R54 to R58, R55 to R59, R56 to R60, R57 to R62, R58 to R64
Connections:
- net SH_A: now also C35.1, C34.1
- net SH_B: now also C51.1, C50.1
- net SH_C: now also C66.1, C65.1
- net V_IN: now also C27.2, C29.2, C31.2, C43.2, C45.2, C47.2, C58.2, C60.2, C62.2, R31.2, R33.2, R47.2, R49.2, R61.2, R63.2
- net at R38.2: now also C41.1, Q6.1 (G), Q8.1 (G), R43.2
- net at C25.1, Q2.1 (G), Q4.1 (G)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: now also R23.2
- net at C56.1, Q10.1 (G), Q12.1 (G)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: now also R53.2
- net at C24.1, Q1.1 (G), Q3.1 (G)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: now also R22.2
- net at C40.1, Q5.1 (G), Q7.1 (G)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: now also R37.2
- net at C55.1, Q11.1 (G), Q9.1 (G)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: now also R52.2
- new net: C34.2, R31.1, R33.1
- new net: C65.2, R61.1, R63.1
- new net: C50.2, R47.1, R49.1
Other:
- note added: "WATT'EVER"
- note removed: "F-Of-C"
- moved on the sheet: C27, C29, C31, C33, C35, C43, C45, C47, C49, C51, C58, C60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

Commit message: Add files via upload
Parts:
- removed C31, C43, C58: 10u @ 100V, Capacitor_SMD:C_2220_5650Metric, symbol BLDC_4-rescue:C-RESCUE-BLDC_4
- removed Q11, Q12, Q3, Q4, Q7, Q8: CSD19536KCS, Package_TO_SOT_THT:TO-220-3_Vertical, symbol Device:Q_NMOS_GDS
- added C27, C28, C29, C30, C32, C34, C45, C46, C47, C48, C50, C52, C62, C63, C64, C65, C67, C69: 100n 100V, Capacitor_SMD:C_0805_2012Metric, symbol Device:C
- added H6, H7: MountingHole_Pad, MountingHole:MountingHole_4mm_Pad_TopOnly, symbol Mechanical:MountingHole_Pad
- C35: renamed from C33; footprint Custom:CP_Radial_D8.0mm_P5.00mm -> Capacitor_THT:CP_Radial_D10.0mm_P5.00mm
- C53: renamed from C49; footprint Custom:CP_Radial_D8.0mm_P5.00mm -> Capacitor_THT:CP_Radial_D10.0mm_P5.00mm
- C70: renamed from C64; footprint Custom:CP_Radial_D8.0mm_P5.00mm -> Capacitor_THT:CP_Radial_D10.0mm_P5.00mm
- renumbered C27 to C31, C29 to C33, C34 to C36, C35 to C37, C36 to C38, C37 to C39, C38 to C40, C39 to C41, C40 to C42, C41 to C43, C42 to C44, C45 to C49, C47 to C51, C50 to C54, C51 to C55, C52 to C56, C53 to C57, C54 to C58, C55 to C59, C56 to C60, C57 to C61, C60 to C66, C62 to C68, C65 to C71, C66 to C72, Q5 to Q3, Q6 to Q4, Q9 to Q5, Q10 to Q6
Connections:
- net GND: now also C27.2, C28.2, C29.2, C30.2, C32.2, C34.2, C45.2, C46.2, C47.2, C48.2, C50.2, C52.2, C62.2, C63.2, C64.2, C65.2, C67.2, C69.2, H7.1
- net V_IN: now also C27.1, C28.1, C29.1, C30.1, C32.1, C34.1, C45.1, C46.1, C47.1, C48.1, C50.1, C52.1, C62.1, C63.1, C64.1, C65.1, C67.1, C69.1, H6.1
Other:
- moved on the sheet: C31, C33, Q1, Q2, Q3, Q4, Q5, Q6

Commit message: Add files via upload
Parts:
- Q1: value NCEP60T20 -> CSD19536KCS
- renumbered R21 to R25, R22 to R26, R23 to R27, R24 to R28, R25 to R29, R26 to R30, R27 to R31, R28 to R32, R29 to R33, R30 to R34, R31 to R35, R32 to R36, R33 to R37, R34 to R38, R35 to R39, R36 to R40, R37 to R41, R38 to R42, R39 to R43, R40 to R44, R41 to R45, R42 to R46, R43 to R47, R44 to R48, R45 to R49, R46 to R50, R47 to R51, R48 to R52, R49 to R53, R50 to R54, R51 to R55, R52 to R56, R53 to R57, R54 to R58, R55 to R59, R56 to R60, R57 to R61, R58 to R62, R59 to R63, R60 to R64, R61 to R65, R62 to R66, R63 to R67, R64 to R68

Commit message: Add files via upload
Parts:
- added D10, D11, D12, D13, D8, D9: 1N5819WS, Diode_SMD:D_SOD-323, symbol Device:D_Schottky
- added Q1, Q10, Q2, Q5, Q6, Q9: MMBT5401, Package_TO_SOT_SMD:SOT-23, symbol Transistor_BJT:MMBTA92
- added R27, R28, R44, R45, R61, R62: 2k2, Resistor_SMD:R_0603_1608Metric, symbol Device:R
- C35: renamed from C24; LCSC C77025 -> C344172
- C36: renamed from C25; LCSC C77025 -> C344172
- C53: renamed from C42; LCSC C77025 -> C344172
- C54: renamed from C43; LCSC C77025 -> C344172
- C70: renamed from C59; LCSC C77025 -> C344172
- C71: renamed from C60; LCSC C77025 -> C344172
- renumbered C21 to C32, C22 to C33, C23 to C34, C26 to C37, C27 to C38, C28 to C39, C29 to C40, C30 to C41, C31 to C42, C32 to C43, C33 to C44, C34 to C45, C35 to C46, C36 to C47, C37 to C48, C38 to C49, C39 to C50, C40 to C51, C41 to C52, C44 to C55, C45 to C56, C46 to C57, C47 to C58, C48 to C59, C49 to C60, C50 to C61, C51 to C62, C52 to C63, C53 to C64, C54 to C65, C55 to C66, C56 to C67, C57 to C68, C58 to C69, C61 to C72, C62 to C73, C63 to C74, C64 to C75, C65 to C76, C66 to C77, C67 to C78, C68 to C79, C69 to C80, C70 to C81, C71 to C82, C72 to C83, Q5 to Q11, Q6 to Q12, Q1 to Q3, Q2 to Q4, Q3 to Q7, Q4 to Q8, R25 to R26, R26 to R29, R27 to R30, R28 to R31, R29 to R32, R32 to R33, R33 to R34, R30 to R35, R31 to R36, R34 to R37, R35 to R38, R36 to R39, R37 to R40, R38 to R41, R39 to R42, R40 to R43, R41 to R46, R42 to R47, R43 to R48, R44 to R49, R45 to R50, R48 to R51, R49 to R52, R46 to R53, R47 to R54, R50 to R55, R51 to R56, R52 to R57, R53 to R58, R54 to R59, R55 to R60, R56 to R63, R57 to R64, R58 to R65, R59 to R66, R62 to R67, R63 to R68, R60 to R69, R61 to R70, R64 to R71, R65 to R72, R66 to R73, R67 to R74, R68 to R75, U6 to U11, U7 to U12, U8 to U13
Connections:
- net SH_A: now also Q1.3 (C)
- net SH_B: now also Q5.3 (C)
- net SH_C: now also Q9.3 (C)
- net at C71.2, NT5.2, Q12.3 (S)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: now also Q10.3 (C)
- net at C71.1, Q12.1 (G), R70.2: now also D13.1 (K), Q10.2 (E); no longer R64.2
- net at C54.2, NT3.2, Q8.3 (S)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: now also Q6.3 (C)
- net at C36.2, NT1.2, Q4.3 (S)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: now also Q2.3 (C)
- net at C54.1, Q8.1 (G), R54.2: now also D11.1 (K), Q6.2 (E); no longer R47.2
- net at C53.1, Q7.1 (G), R53.2: now also D10.1 (K), Q5.2 (E); no longer R46.2
- net at C35.1, Q3.1 (G), R35.2: now also D8.1 (K), Q1.2 (E); no longer R29.2
- net at C70.1, Q11.1 (G), R69.2: now also D12.1 (K), Q9.2 (E); no longer R63.2
- net at C36.1, Q4.1 (G), R36.2: now also D9.1 (K), Q2.2 (E); no longer R30.2
- net CURR_A renamed C_A
- net CURR_B renamed C_B
- net CURR_C renamed C_C
- new net: D10.2 (A), R44.2, R46.2
- new net: D8.2 (A), R27.2, R29.2
- new net: D11.2 (A), R45.2, R47.2
- new net: D12.2 (A), R61.2, R63.2
- new net: Q5.1 (B), R44.1
- new net: Q2.1 (B), R28.1
- new net: D9.2 (A), R28.2, R30.2
- new net: Q9.1 (B), R61.1
- new net: D13.2 (A), R62.2, R64.2
- new net: Q10.1 (B), R62.1
- new net: Q6.1 (B), R45.1
- new net: Q1.1 (B), R27.1
Other:
- note added: "Only reserve room for 2.2nF cap"
- moved on the sheet: C35, C36, C53, C54, C70, C71, R30, R35, R36, R47, R53, R54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

Commit message: Add files via upload
Parts:
- removed C42, C44, C60, C62, C77, C79: 10u @ 100V, Capacitor_SMD:C_2220_5650Metric, symbol BLDC_4-rescue:C-RESCUE-BLDC_4
- removed C46, C64, C81: 470u 80V, Capacitor_THT:CP_Radial_D10.0mm_P5.00mm, symbol Device:C_Polarized_US
- removed H6, H7: MountingHole_Pad, MountingHole:MountingHole_4mm_Pad_TopOnly, symbol Mechanical:MountingHole_Pad
- added C41, C42, C43, C44, C45, C62, C63, C64, C65, C66, C82, C83, C84, C85, C86: 100n 100V, Capacitor_SMD:C_0805_2012Metric, symbol Device:C
- renumbered C32 to C29, C33 to C30, C34 to C31, C35 to C32, C36 to C33, C37 to C34, C38 to C35, C39 to C36, C40 to C37, C41 to C38, C43 to C39, C45 to C40, C47 to C46, C48 to C47, C61 to C60, C63 to C61, C65 to C67, C66 to C68, C67 to C70, C68 to C71, C69 to C72, C70 to C73, C71 to C74, C72 to C75, C73 to C76, C74 to C77, C75 to C78, C76 to C79, C78 to C80, C80 to C81, C82 to C87, C83 to C88, R26 to R23, R27 to R24, R28 to R25, R29 to R26, R30 to R27, R31 to R28, R32 to R29, R33 to R30, R34 to R31, R35 to R32, R36 to R33, R37 to R34, R38 to R35, R39 to R36, R40 to R37, R41 to R38, R42 to R39, R43 to R40, R44 to R41, R45 to R42, R46 to R43, R47 to R44, R48 to R45, R49 to R46, R50 to R47, R51 to R48, R52 to R49, R53 to R50, R54 to R51, R55 to R52, R56 to R53, R57 to R54, R58 to R55, R59 to R56, R60 to R57, R61 to R58, R62 to R59, R63 to R60, R64 to R61, R65 to R62, R66 to R63, R67 to R64, R68 to R65, R69 to R66, R70 to R67, R71 to R68, R72 to R69, R73 to R70, R74 to R71, R75 to R72
Connections:
- net GND: now also C41.2, C42.2, C43.2, C44.2, C45.2, C62.2, C63.2, C64.2, C65.2, C66.2, C82.2, C83.2, C84.2, C85.2, C86.2
- net V_IN: now also C41.1, C42.1, C43.1, C44.1, C45.1, C62.1, C63.1, C64.1, C65.1, C66.1, C82.1, C83.1, C84.1, C85.1, C86.1
- net C_A renamed CURR_A
- net C_B renamed CURR_B
- net C_C renamed CURR_C
Other:
- note added: "FOC KING"
- note added: "Op-Amp, Input-to-Output Coupling To minimize capacitive coupling, the input and output signal traces should not be in parallel. This helps reduce unwanted positive feedback."
- note removed: "WATT'EVER"
- moved on the sheet: C35, C36, C37, C38, C39, C40, C56, C57, C58, C59, C60, C61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

Commit message: Add files via upload
Parts:
- renumbered C49 to C48, C50 to C49, C51 to C50, C52 to C51, C53 to C52, C54 to C53, C55 to C54, C56 to C55, C57 to C56, C58 to C57, C59 to C58, C60 to C59, C61 to C60, C62 to C61, C63 to C62, C64 to C63, C65 to C64, C66 to C65, C67 to C66, C68 to C67, C70 to C68, C71 to C69, C72 to C70, C73 to C71, C74 to C72, C75 to C73, C76 to C74, C77 to C75, C78 to C76, C79 to C77, C80 to C78, C81 to C79, C82 to C80, C83 to C81, C84 to C82, C85 to C83, C86 to C84, C87 to C85, C88 to C86
